File: kicad/xDuinoRailControl/control-board.kicad_sch (KiCad schematic)
At the start: 5 parts, among them J3 OLED_SOCKET, U2 MOUDLE-SEEEDUINO-XIAO-ESP32C3, U3 L78L05_SOT89

Commit message: xDuinoRailControl
Parts:
- removed C1: 1uF, Capacitor_SMD:C_0805_2012Metric_Pad1.18x1.45mm_HandSolder, symbol Device:C
- removed C2: 47uF, Capacitor_SMD:C_0805_2012Metric_Pad1.18x1.45mm_HandSolder, symbol Device:C_Polarized
- removed U3: L78L05_SOT89, Package_TO_SOT_SMD:SOT-89-3, symbol Regulator_Linear:L78L05_SOT89
- added SW1: SW_Nidec_CAS-120A1, Button_Switch_SMD:Nidec_Copal_CAS-120A, symbol Switch:SW_Nidec_CAS-120A1
- J3: LCSC (none) -> C2718488
- U2: value MOUDLE-SEEEDUINO-XIAO-ESP32C3 -> XIAO-ESP32C3
Connections:
- net +5V: no longer J3.3 (Pin_3)
- net GND: now also SW1.1 (C)
- net +3V3: now reaches U2.12 (3V3)
- net +3V3: now also J3.3 (Pin_3), SW1.3 (A)
- net at U2.9 (PA7_A8_D8_SCK): now also SW1.2 (B)
- no-connect marks 6 -> 4
Other:
- moved on the sheet: J3

Commit message: Add encoder
Parts:
- added R4: 10k, symbol Device:R
- added SW2: RotaryEncoder_Switch, Rotary_Encoder:RotaryEncoder_Alps_EC11E-Switch_Vertical_H20mm_CircularMountingHoles, symbol Device:RotaryEncoder_Switch
Connections:
- net +3V3: now also R4.1
- net BRAKE: now also U2.4 (PA11_A3_D3); no longer U2.2 (PA4_A1_D1)
- net GND: now also SW2.S2
- net PWM: now also U2.7 (PB08_A6_D6_TX); no longer U2.1 (PA02_A0_D0)
- net SENSE: now also U2.2 (PA4_A1_D1); no longer U2.4 (PA11_A3_D3)
- net at U2.9 (PA7_A8_D8_SCK): now also SW2.C; no longer SW1.2 (B)
- net at U2.10 (PA5_A9_D9_MISO): now also SW2.A
- net at U2.11 (PA6_A10_D10_MOSI): now also R4.2, SW2.S1
- net at U2.8 (PB09_A7_D7_RX): now also SW2.B
- new net: SW1.2 (B), U2.1 (PA02_A0_D0)
- no-connect marks 4 -> 0
Other:
- moved on the sheet: SW1

Commit message: More improvements
Parts:
- added A1: Arduino_UNO_R3, Module:Arduino_UNO_R3, symbol MCU_Module:Arduino_UNO_R3
- R4: footprint (none) -> Resistor_SMD:R_0805_2012Metric_Pad1.20x1.40mm_HandSolder
- U2: footprint XIAO:MOUDLE14P-SMD-2.54-21X17.8MM -> MOUDLE14P-SMD-2.54-21X17.8MM
Connections:
- net +3V3: now also A1.4 (3V3)
- net +5V: now also A1.5 (+5V)
- net BRAKE: now also A1.24 (D9)
- net DIRECTION: now also A1.27 (D12)
- net GND: now also A1.29 (GND), A1.6 (GND), A1.7 (GND)
- net PWM: now also A1.18 (D3)
- net SCL: now also A1.14 (SCL/A5), A1.32 (SCL/A5)
- net SDA: now also A1.13 (SDA/A4), A1.31 (SDA/A4)
- net SENSE: now also A1.9 (A0)
- net DPU: now reaches R4.2, SW2.S1, U2.11 (PA6_A10_D10_MOSI)
- net DPU: now also A1.20 (D5)
- net DC1: now reaches SW2.A, U2.10 (PA5_A9_D9_MISO)
- net DC1: now also A1.21 (D6)
- net DC3: now reaches SW2.B, U2.8 (PB09_A7_D7_RX)
- net DC3: now also A1.23 (D8)
- net DC2: now reaches SW2.C, U2.9 (PA7_A8_D8_SCK)
- net DC2: now also A1.22 (D7)
- no-connect marks 0 -> 13
