File: kicad/xDuinoRailShield/xDuinoRailShield.kicad_sch (KiCad schematic)
At the start: 0 parts

Commit message: More nice changes
Other:
- sheet Audio Jack 3.5mm renamed Audio Interfaces
- sheet Loco Adapters renamed Connectors 21mtc / PluXX / NEMA
- added sheet Motor and Power drivers (motor-n-power-drivers.kicad_sch)
- sheet Audio Interfaces: file audio_jack.kicad_sch -> audio_interfaces.kicad_sch
- sheet Connectors 21mtc / PluXX / NEMA ports: added AUX1_AMP, AUX2_AMP, AUX3_AMP, AUX[1..8], F0_BACKWARD_AMP, F0_FRONTWARD_AMP, MOTOR_AMP0, MOTOR_AMP1; removed AUX1, AUX2, AUX3, AUX4, AUX5, AUX6, AUX7, AUX8
- sheet Railcom-Feedback ports: added DCC[0..1]; removed DCC_0, DCC_1
