File: kicad/xDuinoRailShield/loco-adapters.kicad_sch (KiCad schematic)
At the start: 5 parts, among them J3 PLUXX22, J4 21mtc, U5 ULN2003A, U6 ULN2003A, U8 DRV8872DDA

Commit message: More nice changes
Parts:
- removed U5, U6: ULN2003A, symbol Transistor_Array:ULN2003A
- removed U8: DRV8872DDA, Package_SO:Texas_HTSOP-8-1EP_3.9x4.9mm_P1.27mm_EP2.95x4.9mm_Mask2.4x3.1mm_ThermalVias, symbol Driver_Motor:DRV8872DDA
- added J5: Conn_02x04_Counter_Clockwise, Connector_PinHeader_2.54mm:PinHeader_2x04_P2.54mm_Vertical_SMD, symbol Connector_Generic:Conn_02x04_Counter_Clockwise
- added J6: 21mtc, Connector_PinSocket_1.27mm:PinSocket_2x11_P1.27mm_Vertical_SMD, symbol Connector_Generic:Conn_02x11_Counter_Clockwise
- added J7: Conn_01x06, symbol Connector_Generic:Conn_01x06
Connections:
- net +5V: now also J6.12 (Pin_12)
- net AUX1_AMP: now also J6.15 (Pin_15)
- net AUX2_AMP: now also J6.14 (Pin_14)
- net AUX3_AMP: now also J6.13 (Pin_13)
- net AUX4: now also J6.4 (Pin_4)
- net AUX5: now also J6.17 (Pin_17)
- net AUX6: now also J6.3 (Pin_3)
- net AUX7: now also J6.1 (Pin_1)
- net AUX8: now also J6.2 (Pin_2)
- net AUX89_ZBCLK: now also J6.5 (Pin_5)
- net AUX910_ZBDATA: now also J6.6 (Pin_6)
- net DCC0: now also J5.8 (Pin_8), J6.21 (Pin_21), J7.4 (Pin_4)
- net DCC1: now also J5.4 (Pin_4), J6.22 (Pin_22), J7.3 (Pin_3)
- net F0_BACKWARD_AMP: now also J5.6 (Pin_6), J6.8 (Pin_8), J7.6 (Pin_6)
- net F0_FRONTWARD_AMP: now also J5.2 (Pin_2), J6.7 (Pin_7), J7.5 (Pin_5)
- net GND: now also J6.20 (Pin_20)
- net MOTOR+: no longer J4.19 (Pin_19)
- net MOTOR-: no longer J4.18 (Pin_18)
- net SPEAKER0: now also J6.10 (Pin_10)
- net SPEAKER1: now also J6.9 (Pin_9)
- net U+: now also J5.7 (Pin_7), J6.16 (Pin_16)
- new net MOTOR_AMP0: J4.18 (Pin_18), J5.1 (Pin_1), J6.18 (Pin_18), J7.1 (Pin_1)
- new net MOTOR_AMP1: J4.19 (Pin_19), J5.5 (Pin_5), J6.19 (Pin_19), J7.2 (Pin_2)
- no-connect marks 2 -> 3
Other:
- moved on the sheet: J3

Commit message: More busses added
Parts:
- removed J6: 21mtc, Connector_PinSocket_1.27mm:PinSocket_2x11_P1.27mm_Vertical_SMD, symbol Connector_Generic:Conn_02x11_Counter_Clockwise
- renumbered J4 to J101, J5 to J102, J3 to J103, J7 to J104
Connections:
- net AUX1_AMP: no longer J101.15 (Pin_15)
- net AUX2_AMP: no longer J101.14 (Pin_14)
- net AUX3_AMP: no longer J101.13 (Pin_13)
- net SPEAKER0: now also J101.9 (Pin_9), J103.15 (Pin_15); no longer J101.10 (Pin_10), J103.17 (Pin_17)
- net SPEAKER1: now also J101.10 (Pin_10), J103.17 (Pin_17); no longer J101.9 (Pin_9), J103.15 (Pin_15)
- net F0_BACKWARD_AMP renamed F0.AMP_BACKWARD
- net F0.AMP_BACKWARD: now also J104.5 (Pin_5); no longer J101.8 (Pin_8), J104.6 (Pin_6)
- removed net F0_FRONTWARD_AMP: J101.7 (Pin_7), J102.2 (Pin_2), J103.7 (Pin_7), J104.5 (Pin_5)
- net MOTOR+ renamed AMP_MOTOR0
- net AMP_MOTOR0: now also J101.18 (Pin_18), J102.1 (Pin_1), J104.2 (Pin_2)
- net MOTOR- renamed AMP_MOTOR1
- net AMP_MOTOR1: now also J101.19 (Pin_19), J102.5 (Pin_5), J104.1 (Pin_1)
- removed net MOTOR_AMP0: J101.18 (Pin_18), J102.1 (Pin_1), J104.1 (Pin_1)
- removed net MOTOR_AMP1: J101.19 (Pin_19), J102.5 (Pin_5), J104.2 (Pin_2)
- new net AMP_AUX1: J101.15 (Pin_15)
- new net AMP_AUX2: J101.14 (Pin_14)
- new net AMP_AUX3: J101.13 (Pin_13)
- new net F0.AMP_FOREWARD: J102.2 (Pin_2), J104.6 (Pin_6)
- new net F0.AMP_FRONTWARD: J103.7 (Pin_7)
- new net F0.BACKWARD_AMP: J101.8 (Pin_8)
- new net F0.FOREWARD_AMP: J101.7 (Pin_7)

Commit message: Draft of loco decoder
Parts:
- added J105: 21mtc_mrkl, Connector_PinSocket_1.27mm:PinSocket_2x11_P1.27mm_Vertical_SMD, symbol Connector_Generic:Conn_02x11_Counter_Clockwise
- J101: value 21mtc -> 21mtc_nema; now not fitted; now left out of the parts list
- J102, J103, J104: now not fitted; now left out of the parts list
Connections:
- net +5V: now also J105.12 (Pin_12)
- net AMP_AUX1: now also J105.15 (Pin_15)
- net AMP_AUX2: now also J105.14 (Pin_14)
- net AMP_AUX3: now also J105.13 (Pin_13)
- net AMP_MOTOR0: now also J105.18 (Pin_18)
- net AMP_MOTOR1: now also J105.19 (Pin_19)
- net AUX4: now also J105.4 (Pin_4)
- net AUX5: now also J105.17 (Pin_17)
- net AUX6: now also J105.3 (Pin_3)
- net AUX7: now also J105.1 (Pin_1)
- net AUX8: now also J105.2 (Pin_2)
- net AUX89_ZBCLK: now also J105.5 (Pin_5)
- net AUX910_ZBDATA: now also J105.6 (Pin_6)
- net DCC0: now also J105.21 (Pin_21)
- net DCC1: now also J105.22 (Pin_22)
- net F0.BACKWARD_AMP: now also J105.8 (Pin_8)
- net F0.FOREWARD_AMP: now also J105.7 (Pin_7)
- net GND: now also J105.20 (Pin_20)
- net SPEAKER0: now also J105.9 (Pin_9)
- net SPEAKER1: now also J105.10 (Pin_10)
- net U+: now also J105.16 (Pin_16)
- no-connect marks 3 -> 4

Commit message: A lot of fixes
Parts:
- removed J105: 21mtc_mrkl, Connector_PinSocket_1.27mm:PinSocket_2x11_P1.27mm_Vertical_SMD, symbol Connector_Generic:Conn_02x11_Counter_Clockwise
- added J106: 21mtc_mrkl, Connector_PinSocket_1.27mm:PinSocket_2x11_P1.27mm_Vertical_SMD, symbol Connector_Generic:Conn_02x11_Odd_Even
- added JP101, JP102, JP103, JP104, JP105, JP106: SolderJumper_2_Bridged, Jumper:SolderJumper-2_P1.3mm_Bridged_Pad1.0x1.5mm, symbol Jumper:SolderJumper_2_Bridged
- renumbered J104 to J105
Connections:
- net AUX1_AMP is gone; now on net AMP_AUX1: J103.16 (Pin_16)
- net AUX2_AMP is gone; now on net AMP_AUX2: J103.18 (Pin_18)
- net AUX3_AMP is gone; now on net AMP_AUX2: J103.2 (Pin_2)
- net F0.FOREWARD_AMP is gone; now on net AMP_FUNC0: J101.7 (Pin_7)
- net +5V: now also J106.22 (Pin_22)
- net AMP_AUX1: now also J106.16 (Pin_16)
- net AMP_AUX2: now also J106.18 (Pin_18)
- net AMP_AUX3: now also J106.20 (Pin_20)
- net AMP_MOTOR0: now also J106.10 (Pin_10), JP103.2 (B)
- net AMP_MOTOR1: now also J106.8 (Pin_8), JP104.2 (B)
- net AUX4: now also J106.7 (Pin_7)
- net AUX5: now also J106.12 (Pin_12)
- net AUX6: now also J106.5 (Pin_5)
- net AUX7: now also J106.1 (Pin_1)
- net AUX8: now also J106.3 (Pin_3)
- net AUX89_ZBCLK: now also J106.9 (Pin_9)
- net AUX910_ZBDATA: now also J106.11 (Pin_11)
- net DCC0: now also J106.4 (Pin_4), JP101.2 (B)
- net DCC1: now also J106.2 (Pin_2), JP102.2 (B)
- net GND: now also J106.6 (Pin_6)
- net SPEAKER0: now also J106.17 (Pin_17)
- net SPEAKER1: now also J106.19 (Pin_19)
- net U+: now also J106.14 (Pin_14)
- net AUX4_AMP renamed AMP_AUX4
- net AUX5_AMP renamed AMP_AUX5
- net AUX6_AMP renamed AMP_AUX6
- net AUX7_AMP renamed AMP_AUX7
- net F0.AMP_BACKWARD renamed FUNC1
- net FUNC1: now also JP106.2 (B); no longer J103.13 (Pin_13)
- net F0.AMP_FOREWARD renamed FUNC0
- net FUNC0: now also JP105.2 (B)
- net F0.AMP_FRONTWARD renamed AMP_FUNC0
- net AMP_FUNC0: now also J106.13 (Pin_13)
- net F0.BACKWARD_AMP renamed AMP_FUNC1
- net AMP_FUNC1: now also J103.13 (Pin_13), J106.15 (Pin_15)
- no-connect marks 4 -> 10
Other:
- note added: "21mtc header (Märklin)"
- note added: "21mtc header (NEM660)"
- note added: "6-pin (NEM651)"
- note added: "8-pin (NEM652)"
- note added: "Bus extraction"
- note added: "Copper Pads"
- note added: "pluxx22 (NEM658)"
