File: kicad/xDuinoRailShield/io-carrier-board.kicad_sch (KiCad schematic)
At the start: 8 parts, among them J601 Screw_Terminal_01x02, U601 MOUDLE-SEEEDUINO-XIAO-ESP32C3

Commit message: A lot of fixes
Parts:
- added D503: LED, LED_SMD:LED_0805_2012Metric_Pad1.15x1.40mm_HandSolder, symbol Device:LED
- added R503: 1k, Resistor_SMD:R_0805_2012Metric_Pad1.20x1.40mm_HandSolder, symbol Device:R
- R501: renamed from R602; footprint Resistor_SMD:R_0603_1608Metric_Pad0.98x0.95mm_HandSolder -> Resistor_SMD:R_0805_2012Metric_Pad1.20x1.40mm_HandSolder
- R502: renamed from R601; footprint Resistor_SMD:R_0603_1608Metric_Pad0.98x0.95mm_HandSolder -> Resistor_SMD:R_0805_2012Metric_Pad1.20x1.40mm_HandSolder
- renumbered A601 to A501, D602 to D501, D601 to D502, J601 to J501, JP601 to JP501, U601 to U501
Connections:
- net +5V: now also D503.1 (K)
- net ANALOG_5V: no longer U501.2 (A1)
- net AUX2: no longer U501.6 (SDA_A5)
- net AUX3: no longer U501.7 (SCL_A6)
- net DAC: no longer U501.1 (A0)
- net GND: now also R503.1
- net +3V3: now reaches U501.12 (3V3)
- net +3V3: now also A501.4 (3V3)
- net EMF_MOTOR0: now reaches A501.10 (A1)
- net EMF_MOTOR0: now also U501.1 (A0)
- net I2C.SDA: now reaches A501.13 (SDA/A4)
- net I2C.SCL: now reaches A501.14 (SCL/A5)
- net F0.BACKWARD renamed FUNC0
- net FUNC0: now also A501.27 (D12); no longer A501.28 (D13)
- net F0.FOREWARD renamed FUNC1
- net FUNC1: now also A501.28 (D13); no longer A501.27 (D12)
- new net: D503.2 (A), R503.2
- new net EMF_MOTOR1: U501.2 (A1)
- new net I2C0: U501.7 (SCL_A6)
- new net I2C1: U501.6 (SDA_A5)
- no-connect marks 14 -> 9
Other:
- note added: "Arduino Shield"
- note added: "Screw Terminal & DCC-LEDs"
- note added: "XIAO Shield"
- moved on the sheet: D501, D502, J501, R501, R502, U501

Commit message: Final version
Parts:
- removed D503: LED, LED_SMD:LED_0805_2012Metric_Pad1.15x1.40mm_HandSolder, symbol Device:LED
- removed R503: 1k, Resistor_SMD:R_0805_2012Metric_Pad1.20x1.40mm_HandSolder, symbol Device:R

Commit message: More refactoring
Other:
- added sheet RP2040-OnBoard (rp2040-onboard.kicad_sch)
- moved on the sheet: D501, D502, J501, R501, R502
Changed lines of the file:
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@@
 	)
 	(junction
-		(at 198.12 71.12)
+		(at 218.44 66.04)
 		(diameter 0)
 		(color 0 0 0 0)
@@
 	)
 	(junction
-		(at 198.12 52.07)
+		(at 218.44 46.99)
 		(diameter 0)
 		(color 0 0 0 0)
@@
 	(wire
 		(pts
-			(xy 198.12 52.07) (xy 198.12 53.34)
-		)
-		(stroke
-			(width 0)
-			(type default)
-		)
-	)
-	(wire
-		(pts
-			(xy 190.5 52.07) (xy 198.12 52.07)
+			(xy 218.44 46.99) (xy 218.44 48.26)
+		)
+		(stroke
+			(width 0)
+			(type default)
+		)
+	)
+	(wire
+		(pts
+			(xy 210.82 46.99) (xy 218.44 46.99)
 		)
 		(stroke
@@
 	(wire
 		(pts
-			(xy 198.12 71.12) (xy 198.12 68.58)
+			(xy 218.44 66.04) (xy 218.44 63.5)
 		)
 		(stroke
@@
 	(wire
 		(pts
-			(xy 190.5 71.12) (xy 190.5 69.85)
+			(xy 210.82 66.04) (xy 210.82 64.77)
 		)
 		(stroke
@@
 	(wire
 		(pts
-			(xy 190.5 52.07) (xy 190.5 54.61)
+			(xy 210.82 46.99) (xy 210.82 49.53)
 		)
 		(stroke
@@
 	(wire
 		(pts
-			(xy 213.36 54.61) (xy 213.36 71.12)
+			(xy 233.68 49.53) (xy 233.68 66.04)
 		)
 		(stroke
@@
 	(wire
 		(pts
-			(xy 223.52 52.07) (xy 198.12 52.07)
+			(xy 243.84 46.99) (xy 218.44 46.99)
 		)
 		(stroke
@@
 	(wire
 		(pts
-			(xy 223.52 54.61) (xy 213.36 54.61)
+			(xy 243.84 49.53) (xy 233.68 49.53)
 		)
 		(stroke
@@
 	(wire
 		(pts
-			(xy 213.36 71.12) (xy 198.12 71.12)
+			(xy 233.68 66.04) (xy 218.44 66.04)
 		)
 		(stroke
@@
 	(wire
 		(pts
-			(xy 198.12 71.12) (xy 190.5 71.12)
+			(xy 218.44 66.04) (xy 210.82 66.04)
 		)
 		(stroke
@@
 	(text "Screw Terminal & DCC-LEDs"
 		(exclude_from_sim no)
-		(at 214.63 44.196 0)
+		(at 234.95 39.116 0)
 		(effects
 			(font
@@
 	)
 	(label "DCC0"
-		(at 222.25 52.07 180)
+		(at 242.57 46.99 180)
 		(fields_autoplaced yes)
 		(effects
@@
 	)
 	(label "DCC1"
-		(at 222.25 54.61 180)
+		(at 242.57 49.53 180)
 		(fields_autoplaced yes)
 		(effects
@@
 	(hierarchical_label "DCC[0..1]"
 		(shape bidirectional)
-		(at 236.22 53.34 0)
+		(at 256.54 48.26 0)
 		(fields_autoplaced yes)
 		(effects
@@
 	(symbol
 		(lib_id "Device:LED")
-		(at 198.12 64.77 90)
+		(at 218.44 59.69 90)
 		(unit 1)
 		(exclude_from_sim yes)
@@
 		(dnp yes)
 		(property "Reference" "D502"
-			(at 201.93 65.0875 90)
+			(at 222.25 60.0075 90)
 			(effects
 				(font
@@
 		)
 		(property "Value" "LED"
-			(at 201.93 67.6275 90)
+			(at 222.25 62.5475 90)
 			(effects
 				(font
@@
 		)
 		(property "Footprint" "LED_SMD:LED_0805_2012Metric_Pad1.15x1.40mm_HandSolder"
-			(at 198.12 64.77 0)
+			(at 218.44 59.69 0)
 			(effects
 				(font
@@
 		)
 		(property "Datasheet" "~"
-			(at 198.12 64.77 0)
+			(at 218.44 59.69 0)
 			(effects
 				(font
@@
 		)
 		(property "Description" "Light emitting diode"
-			(at 198.12 64.77 0)
+			(at 218.44 59.69 0)
 			(effects
 				(font
@@
 		)
 		(property "LCSC" "C2297"
-			(at 198.12 64.77 0)
+			(at 218.44 59.69 0)
 			(effects
 				(font
@@
 		)
 		(property "Field-1" ""
-			(at 198.12 64.77 0)
+			(at 218.44 59.69 0)
 			(effects
 				(font
@@
 	(symbol
 		(lib_id "Device:R")
-		(at 198.12 57.15 0)
+		(at 218.44 52.07 0)
 		(unit 1)
 		(exclude_from_sim yes)
@@
 		(dnp yes)
 		(property "Reference" "R502"
-			(at 200.66 55.88 0)
+			(at 220.98 50.8 0)
 			(effects
 				(font
@@
 		)
 		(property "Value" "3k3"
-			(at 200.66 58.42 0)
+			(at 220.98 53.34 0)
 			(effects
 				(font
@@
 		)
 		(property "Footprint" "Resistor_SMD:R_0805_2012Metric_Pad1.20x1.40mm_HandSolder"
-			(at 196.342 57.15 90)
+			(at 216.662 52.07 90)
 			(effects
 				(font
@@
 		)
 		(property "Datasheet" "~"
-			(at 198.12 57.15 0)
+			(at 218.44 52.07 0)
 			(effects
 				(font
@@
 		)
 		(property "Description" "Resistor"
-			(at 198.12 57.15 0)
+			(at 218.44 52.07 0)
 			(effects
 				(font
@@
 		)
 		(property "LCSC" "C26010"
-			(at 198.12 57.15 0)
+			(at 218.44 52.07 0)
 			(effects
 				(font
@@
 		)
 		(property "Field-1" ""
-			(at 198.12 57.15 0)
+			(at 218.44 52.07 0)
 			(effects
 				(font
@@
 	(symbol
 		(lib_id "Device:R")
-		(at 190.5 66.04 180)
+		(at 210.82 60.96 180)
 		(unit 1)
 		(exclude_from_sim yes)
@@
 		(dnp yes)
 		(property "Reference" "R501"
-			(at 187.96 67.31 0)
+			(at 208.28 62.23 0)
 			(effects
 				(font
@@
 		)
 		(property "Value" "3k3"
-			(at 187.96 64.77 0)
+			(at 208.28 59.69 0)
 			(effects
 				(font
@@
 		)
 		(property "Footprint" "Resistor_SMD:R_0805_2012Metric_Pad1.20x1.40mm_HandSolder"
-			(at 192.278 66.04 90)
+			(at 212.598 60.96 90)
 			(effects
 				(font
@@
 		)
 		(property "Datasheet" "~"
-			(at 190.5 66.04 0)
+			(at 210.82 60.96 0)
 			(effects
 				(font
@@
 		)
 		(property "Description" "Resistor"
-			(at 190.5 66.04 0)
+			(at 210.82 60.96 0)
 			(effects
 				(font
@@
 		)
 		(property "LCSC" "C26010"
-			(at 190.5 66.04 0)
+			(at 210.82 60.96 0)
 			(effects
 				(font
@@
 		)
 		(property "Field-1" ""
-			(at 190.5 66.04 0)
+			(at 210.82 60.96 0)
 			(effects
 				(font
@@
 	(symbol
 		(lib_id "Connector:Screw_Terminal_01x02")
-		(at 228.6 54.61 0)
+		(at 248.92 49.53 0)
 		(mirror x)
 		(unit 1)
@@
 		(dnp yes)
 		(property "Reference" "J501"
-			(at 228.6 57.15 0)
+			(at 248.92 52.07 0)
 			(effects
 				(font
@@
 		)
 		(property "Value" "Screw_Terminal_01x02"
-			(at 209.55 59.69 0)
+			(at 229.87 54.61 0)
 			(effects
 				(font
@@
 		)
 		(property "Footprint" "TerminalBlock:TerminalBlock_bornier-2_P5.08mm"
-			(at 228.6 54.61 0)
+			(at 248.92 49.53 0)
 			(effects
 				(font
@@
 		)
 		(property "Datasheet" "~"
-			(at 228.6 54.61 0)
+			(at 248.92 49.53 0)
 			(effects
 				(font
@@
 		)
 		(property "Description" "Generic screw terminal, single row, 01x02, script generated (kicad-library-utils/schlib/autogen/connector/)"
-			(at 228.6 54.61 0)
+			(at 248.92 49.53 0)
 			(effects
 				(font
@@
 		)
 		(property "LCSC" "C8269"
-			(at 228.6 54.61 0)
+			(at 248.92 49.53 0)
 			(effects
 				(font
@@
 		)
 		(property "Field-1" ""
-			(at 228.6 54.61 0)
+			(at 248.92 49.53 0)
 			(effects
 				(font
@@
 	(symbol
 		(lib_id "Device:LED")
-		(at 190.5 58.42 270)
+		(at 210.82 53.34 270)
 		(unit 1)
 		(exclude_from_sim yes)
@@
 		(dnp yes)
 		(property "Reference" "D501"
-			(at 186.69 58.1025 90)
+			(at 207.01 53.0225 90)
 			(effects
 				(font
@@
 		)
 		(property "Value" "LED"
-			(at 186.69 55.5625 90)
+			(at 207.01 50.4825 90)
 			(effects
 				(font
@@
 		)
 		(property "Footprint" "LED_SMD:LED_0805_2012Metric_Pad1.15x1.40mm_HandSolder"
-			(at 190.5 58.42 0)
+			(at 210.82 53.34 0)
 			(effects
 				(font
@@
 		)
 		(property "Datasheet" "~"
-			(at 190.5 58.42 0)
+			(at 210.82 53.34 0)
 			(effects
 				(font
@@
 		)
 		(property "Description" "Light emitting diode"
-			(at 190.5 58.42 0)
+			(at 210.82 53.34 0)
 			(effects
 				(font
@@
 		)
 		(property "LCSC" "C2297"
-			(at 190.5 58.42 0)
+			(at 210.82 53.34 0)
 			(effects
 				(font
@@
 		)
 		(property "Field-1" ""
-			(at 190.5 58.42 0)
+			(at 210.82 53.34 0)
 			(effects
 				(font
@@
 				)
 			)
+		)
+	)
+	(sheet
+		(at 213.36 96.52)
+		(size 54.61 48.26)
+		(fields_autoplaced yes)
+		(stroke
+			(width 0.1524)
+			(type solid)
+		)
+		(fill
+			(color 0 0 0 0.0000)
+		)
+		(property "Sheetname" "RP2040-OnBoard"
+			(at 213.36 95.8084 0)
+			(effects
+				(font
+					(size 1.27 1.27)
+				)
+				(justify left bottom)
+			)
+		)
+		(property "Sheetfile" "rp2040-onboard.kicad_sch"
+			(at 213.36 145.3646 0)
+			(effects
+				(font
+					(size 1.27 1.27)
+				)
+				(justify left top)
+			)
+		)
+		(instances
+			(project "xDuinoRailShield"
+				(path "/e63e39d7-6ac0-4ffd-8aa3-1841a4541b55/73623b68-3f11-49c2-b33b-f7aef9e34c5f"
+					(page "11")
+				)
+			)
