File: kicad/xDuinoRailShield/rails_power_dc-dc-ldo-5v.kicad_sch (KiCad schematic)
At the start: 17 parts, among them U701 L78L05_SOT89, U702 TPS5430DDA

Commit message: More refactoring
Parts:
- removed U701: L78L05_SOT89, Package_TO_SOT_SMD:SOT-89-3, symbol Regulator_Linear:L78L05_SOT89
- added C708: 1uF, Capacitor_SMD:C_0402_1005Metric_Pad0.74x0.62mm_HandSolder, symbol Device:C
- added C709: 47uF, Capacitor_SMD:C_0805_2012Metric_Pad1.18x1.45mm_HandSolder, symbol Device:C_Polarized
- added D501, D502, D503, D504: SS54, Diode_SMD:D_SMA, symbol Device:D
- added U701: HT7533-1, Package_TO_SOT_SMD:SOT-89-3, symbol Regulator_Linear:L78L33_SOT89
- added U703: L78L05_SOT89, Package_TO_SOT_SMD:SOT-89-3, symbol Regulator_Linear:L78L05_SOT89
- C702: LCSC C28323 -> C52923
- C705: footprint Capacitor_SMD:C_0402_1005Metric_Pad0.74x0.62mm_HandSolder -> Capacitor_SMD:C_0805_2012Metric_Pad1.18x1.45mm_HandSolder
- D701, D702, D703, D704: LCSC C8678 -> C191023; now not fitted; now left out of the parts list
Connections:
- net +5V: now also C709.1, U703.1 (OUT); no longer C705.1
- net DCC0: now also D501.1 (K), D502.2 (A)
- net DCC1: now also D503.1 (K), D504.2 (A)
- net DCC_VIN: now also C708.1, D502.1 (K), D504.1 (K), U701.3 (IN), U703.3 (IN)
- net GND: now also C708.2, C709.2, D501.2 (A), D503.2 (A), U701.2 (GND), U703.2 (GND)
- new net +3V3: C705.1, U701.1 (OUT)
Other:
- note added: "Bridge Rectifier heavy"
- note added: "Bridge Rectifier light"
- note added: "DC-DC voltage regulator 3.3V"
- note added: "DC-DC voltage regulator 5V"
- note removed: "Bridge Rectifier"
- note removed: "DC-DC voltage regulator"
