File: kicad/xDuinoRailShield/rails_signal_feedback_dcc-railcom-8x50_3v3.kicad_sch (KiCad schematic)
At the start: 9 parts, among them Q401 S8050, Q402 S8550, Q403 S8550, Q404 S8050

Commit message: More refactoring
Parts:
- added R404, R405, R406: 10R, Resistor_SMD:R_0805_2012Metric_Pad1.20x1.40mm_HandSolder, symbol Device:R
- added TP101, TP102, TP103, TP104: TestPoint, TestPoint:TestPoint_Pad_D2.0mm, symbol Connector:TestPoint
- R7: footprint Resistor_SMD:R_0402_1005Metric_Pad0.72x0.64mm_HandSolder -> Resistor_SMD:R_0805_2012Metric_Pad1.20x1.40mm_HandSolder; LCSC C17414 -> C25744
- R8: value 20 -> 15R; footprint Resistor_SMD:R_0402_1005Metric_Pad0.72x0.64mm_HandSolder -> Resistor_SMD:R_0603_1608Metric_Pad0.98x0.95mm_HandSolder; LCSC C17544 -> C22950; now not fitted; now left out of the parts list
- R9: value 6k8 -> 10k; footprint Resistor_SMD:R_0402_1005Metric_Pad0.72x0.64mm_HandSolder -> Resistor_SMD:R_0805_2012Metric_Pad1.20x1.40mm_HandSolder; LCSC C17772 -> C25744
Connections:
- net DCC0: now also TP104.1
- net DCC1: now also D401.2 (A); no longer D401.1 (K)
- net RAILCOM_DATA: now also TP102.1
- net RC_CURR: now also R404.1, R405.1, TP101.1
- net RC_SIGNAL: now also D401.1 (K), TP103.1; no longer D401.2 (A)
- net +5V renamed +3V3
- net +3V3: now also R406.2
- new net: R404.2, R405.2, R406.1
Other:
- note added: "https://normen.railcommunity.de/RCN-217.pdf"
- moved on the sheet: D401, JP401, Q401, Q402, Q403, Q404, R7, R9
