File: kicad/xDuinoRailShield/audio-35jack.kicad_sch (KiCad schematic)
At the start: 3 parts, among them J2 AudioJack2_Ground

Commit message: More stuff
Parts:
- added R1401, R1402: 10k, Resistor_SMD:R_0805_2012Metric_Pad1.20x1.40mm_HandSolder, symbol Device:R
- C1401: renamed from C9; footprint (none) -> Capacitor_SMD:C_1206_3216Metric_Pad1.33x1.80mm_HandSolder; OLI_ID (none) -> 100uf_1206
- J1401: renamed from J2; now not fitted
- RV1401: renamed from RV1; value 10K -> 10k; footprint Potentiometer_SMD:Potentiometer_ACP_CA6-VSMD_Vertical -> Resistor_SMD:R_0805_2012Metric_Pad1.20x1.40mm_HandSolder; OLI_ID (none) -> 10k_0805; now not fitted; now left out of the parts list
Connections:
- net DAC_IN: now also R1401.1
- net GND: now also R1402.2
- net at C1401.1, RV1401.2: now also R1401.2, R1402.1
Other:
- moved on the sheet: C1401
