File: kicad/xDuinoRailShield/i2c-audio-ic.kicad_sch (KiCad schematic)
At the start: 6 parts, among them J201 AudioJack2_Ground, J202 Conn_01x04, J203 Conn_01x05, U201 MCP4725xxx-xCH

Commit message: More refactoring
Connections:
- net SPEAKER0 renamed SPEAKER1
Other:
- moved on the sheet: J202, J203

Commit message: More stuff
Parts:
- removed C201: 100uF, symbol Device:C_Polarized
- removed J201: AudioJack2_Ground, Connector_Audio:Jack_3.5mm_CUI_SJ-3523-SMT_Horizontal, symbol Connector_Audio:AudioJack2_Ground
- removed J202: Conn_01x04, symbol Connector_Generic:Conn_01x04
- removed J203: Conn_01x05, symbol Connector_Generic:Conn_01x05
- removed RV201: 10K, Potentiometer_SMD:Potentiometer_ACP_CA6-VSMD_Vertical, symbol Device:R_Potentiometer
- U501: renamed from U201; footprint Package_TO_SOT_SMD:SOT-23-6_Handsoldering -> Package_TO_SOT_SMD:SOT-23-6; OLI_ID (none) -> MCP4725_SOT-23-6
Other:
- note added: "I2C Audio DAC"
- note removed: "Audio Jack 3.5mm"
- note removed: "SUSI 4-pin"
- note removed: "SUSI 5-pin"
- note removed: "https://normen.railcommunity.de/RCN-600.pdf https://normen.railcommunity.de/RCN-601.pdf"
- moved on the sheet: U501
