File: kicad/xDuinoRailShield/i2c-sensors-gyro-accelerometer.kicad_sch (KiCad schematic)
At the start: 3 parts, among them U901 LIS3MDL, U902 LIS3DH

Commit message: More stuff
Parts:
- C701: renamed from C901; footprint (none) -> Capacitor_SMD:C_0805_2012Metric_Pad1.18x1.45mm_HandSolder; OLI_ID (none) -> 100nF_0805
- U702: renamed from U902; OLI_ID (none) -> LIS3DH_LGA-16
- renumbered U901 to U701
Changed lines of the file:
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@@
 	(version 20231120)
 	(generator "eeschema")
-	(generator_version "7.99")
+	(generator_version "8.0")
 	(paper "A4")
 	(junction
@@
 		(dnp no)
 		(fields_autoplaced yes)
-		(property "Reference" "#PWR0903"
+		(property "Reference" "#PWR0703"
 			(at 78.74 50.8 0)
 			(effects
@@
 		)
 		(instances
+			(project "xDuinoRail-Debug"
+				(path "/3fe1c7d3-674a-46fe-b8de-0718a52fef91/a9360f8b-b1cc-42f1-9c21-011e70a7c774"
+					(reference "#PWR0703")
+					(unit 1)
+				)
+			)
 			(project "xDuinoRailShield"
 				(path "/e63e39d7-6ac0-4ffd-8aa3-1841a4541b55/0bfd6d18-10ce-426c-863e-9c05fb8adf3f"
-					(reference "#PWR0903")
+					(reference "#PWR?")
 					(unit 1)
 				)
@@
 		(dnp no)
 		(fields_autoplaced yes)
-		(property "Reference" "#PWR0907"
+		(property "Reference" "#PWR0707"
 			(at 166.37 49.53 0)
 			(effects
@@
 		)
 		(instances
+			(project "xDuinoRail-Debug"
+				(path "/3fe1c7d3-674a-46fe-b8de-0718a52fef91/a9360f8b-b1cc-42f1-9c21-011e70a7c774"
+					(reference "#PWR0707")
+					(unit 1)
+				)
+			)
 			(project "xDuinoRailShield"
 				(path "/e63e39d7-6ac0-4ffd-8aa3-1841a4541b55/0bfd6d18-10ce-426c-863e-9c05fb8adf3f"
-					(reference "#PWR0907")
+					(reference "#PWR?")
 					(unit 1)
 				)
@@
 		(dnp no)
 		(fields_autoplaced yes)
-		(property "Reference" "U902"
+		(property "Reference" "U702"
 			(at 166.0241 78.74 0)
 			(effects
@@
 			)
 		)
+		(property "OLI_ID" "LIS3DH_LGA-16"
+			(at 163.83 63.5 0)
+			(effects
+				(font
+					(size 1.27 1.27)
+				)
+				(hide yes)
+			)
+		)
 		(pin "14"
 		)
@@
 		)
 		(instances
+			(project "xDuinoRail-Debug"
+				(path "/3fe1c7d3-674a-46fe-b8de-0718a52fef91/a9360f8b-b1cc-42f1-9c21-011e70a7c774"
+					(reference "U702")
+					(unit 1)
+				)
+			)
 			(project "xDuinoRailShield"
 				(path "/e63e39d7-6ac0-4ffd-8aa3-1841a4541b55/0bfd6d18-10ce-426c-863e-9c05fb8adf3f"
-					(reference "U902")
+					(reference "U?")
 					(unit 1)
 				)
@@
 		(dnp no)
 		(fields_autoplaced yes)
-		(property "Reference" "#PWR0901"
+		(property "Reference" "#PWR0701"
 			(at 46.99 63.5 0)
 			(effects
@@
 		)
 		(instances
+			(project "xDuinoRail-Debug"
+				(path "/3fe1c7d3-674a-46fe-b8de-0718a52fef91/a9360f8b-b1cc-42f1-9c21-011e70a7c774"
+					(reference "#PWR0701")
+					(unit 1)
+				)
+			)
 			(project "xDuinoRailShield"
 				(path "/e63e39d7-6ac0-4ffd-8aa3-1841a4541b55/0bfd6d18-10ce-426c-863e-9c05fb8adf3f"
-					(reference "#PWR0901")
+					(reference "#PWR?")
 					(unit 1)
 				)
@@
 		(dnp yes)
 		(fields_autoplaced yes)
-		(property "Reference" "C901"
+		(property "Reference" "C701"
 			(at 96.52 59.69 90)
 			(effects
@@
 			)
 		)
-		(property "Footprint" ""
+		(property "Footprint" "Capacitor_SMD:C_0805_2012Metric_Pad1.18x1.45mm_HandSolder"
 			(at 100.33 66.3448 0)
 			(effects
@@
 			)
 		)
+		(property "OLI_ID" "100nF_0805"
+			(at 96.52 67.31 0)
+			(effects
+				(font
+					(size 1.27 1.27)
+				)
+				(hide yes)
+			)
+		)
 		(pin "2"
 		)
@@
 		)
 		(instances
+			(project "xDuinoRail-Debug"
+				(path "/3fe1c7d3-674a-46fe-b8de-0718a52fef91/a9360f8b-b1cc-42f1-9c21-011e70a7c774"
+					(reference "C701")
+					(unit 1)
+				)
+			)
 			(project "xDuinoRailShield"
 				(path "/e63e39d7-6ac0-4ffd-8aa3-1841a4541b55/0bfd6d18-10ce-426c-863e-9c05fb8adf3f"
-					(reference "C901")
+					(reference "C?")
 					(unit 1)
 				)
@@
 		(dnp no)
 		(fields_autoplaced yes)
-		(property "Reference" "#PWR0902"
+		(property "Reference" "#PWR0702"
 			(at 76.2 87.63 0)
 			(effects
@@
 		)
 		(instances
+			(project "xDuinoRail-Debug"
+				(path "/3fe1c7d3-674a-46fe-b8de-0718a52fef91/a9360f8b-b1cc-42f1-9c21-011e70a7c774"
+					(reference "#PWR0702")
+					(unit 1)
+				)
+			)
 			(project "xDuinoRailShield"
 				(path "/e63e39d7-6ac0-4ffd-8aa3-1841a4541b55/0bfd6d18-10ce-426c-863e-9c05fb8adf3f"
-					(reference "#PWR0902")
+					(reference "#PWR?")
 					(unit 1)
 				)
@@
 		(dnp yes)
 		(fields_autoplaced yes)
-		(property "Reference" "U901"
+		(property "Reference" "U701"
 			(at 78.3941 77.47 0)
 			(effects
@@
 		)
 		(instances
+			(project "xDuinoRail-Debug"
+				(path "/3fe1c7d3-674a-46fe-b8de-0718a52fef91/a9360f8b-b1cc-42f1-9c21-011e70a7c774"
+					(reference "U701")
+					(unit 1)
+				)
+			)
 			(project "xDuinoRailShield"
 				(path "/e63e39d7-6ac0-4ffd-8aa3-1841a4541b55/0bfd6d18-10ce-426c-863e-9c05fb8adf3f"
-					(reference "U901")
+					(reference "U?")
 					(unit 1)
 				)
@@
 		(dnp no)
 		(fields_autoplaced yes)
-		(property "Reference" "#PWR0904"
+		(property "Reference" "#PWR0704"
 			(at 102.87 77.47 0)
 			(effects
@@
 		)
 		(instances
+			(project "xDuinoRail-Debug"
+				(path "/3fe1c7d3-674a-46fe-b8de-0718a52fef91/a9360f8b-b1cc-42f1-9c21-011e70a7c774"
+					(reference "#PWR0704")
+					(unit 1)
+				)
+			)
 			(project "xDuinoRailShield"
 				(path "/e63e39d7-6ac0-4ffd-8aa3-1841a4541b55/0bfd6d18-10ce-426c-863e-9c05fb8adf3f"
-					(reference "#PWR0904")
+					(reference "#PWR?")
 					(unit 1)
 				)
@@
 		(dnp no)
 		(fields_autoplaced yes)
-		(property "Reference" "#PWR0905"
+		(property "Reference" "#PWR0705"
 			(at 133.35 71.12 0)
 			(effects
@@
 		)
 		(instances
+			(project "xDuinoRail-Debug"
+				(path "/3fe1c7d3-674a-46fe-b8de-0718a52fef91/a9360f8b-b1cc-42f1-9c21-011e70a7c774"
+					(reference "#PWR0705")
+					(unit 1)
+				)
+			)
 			(project "xDuinoRailShield"
 				(path "/e63e39d7-6ac0-4ffd-8aa3-1841a4541b55/0bfd6d18-10ce-426c-863e-9c05fb8adf3f"
-					(reference "#PWR0905")
+					(reference "#PWR?")
 					(unit 1)
 				)
@@
 		(dnp no)
 		(fields_autoplaced yes)
-		(property "Reference" "#PWR0906"
+		(property "Reference" "#PWR0706"
 			(at 163.83 87.63 0)
 			(effects
@@
 		)
 		(instances
+			(project "xDuinoRail-Debug"
+				(path "/3fe1c7d3-674a-46fe-b8de-0718a52fef91/a9360f8b-b1cc-42f1-9c21-011e70a7c774"
+					(reference "#PWR0706")
+					(unit 1)
+				)
+			)
 			(project "xDuinoRailShield"
 				(path "/e63e39d7-6ac0-4ffd-8aa3-1841a4541b55/0bfd6d18-10ce-426c-863e-9c05fb8adf3f"
-					(reference "#PWR0906")
-					(unit 1)
-				)
+					(reference "#PWR?")
+					(unit 1)
+				)
