File: kicad/xDuinoRailShield/loco-adapter-maerklin-21mtc.kicad_sch (KiCad schematic)
At the start: 1 part, among them J106 21mtc_mrkl

Commit message: More refactoring
Parts:
- renumbered J106 to J301
Changed lines of the file:
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@@
+		)
+	)
+	(hierarchical_label "AMP_MOTOR[0..1]"
+		(shape input)
+		(at 54.61 38.1 180)
+		(fields_autoplaced yes)
+		(effects
+			(font
+				(size 1.27 1.27)
+			)
+			(justify right)
 		)
 	)
@@
 		)
 	)
+	(hierarchical_label "AUX[1..8]"
+		(shape input)
+		(at 54.61 49.53 180)
+		(fields_autoplaced yes)
+		(effects
+			(font
+				(size 1.27 1.27)
+			)
+			(justify right)
+		)
+	)
+	(hierarchical_label "+3V3"
+		(shape input)
+		(at 90.17 74.93 90)
+		(fields_autoplaced yes)
+		(effects
+			(font
+				(size 1.27 1.27)
+			)
+			(justify left)
+		)
+	)
+	(hierarchical_label "U+"
+		(shape input)
+		(at 86.36 74.93 90)
+		(fields_autoplaced yes)
+		(effects
+			(font
+				(size 1.27 1.27)
+			)
+			(justify left)
+		)
+	)
 	(hierarchical_label "AMP_AUX[1..7]"
 		(shape input)
 		(at 54.61 53.34 180)
-		(fields_autoplaced yes)
-		(effects
-			(font
-				(size 1.27 1.27)
-			)
-			(justify right)
-		)
-	)
-	(hierarchical_label "+3V3"
-		(shape input)
-		(at 90.17 74.93 90)
-		(fields_autoplaced yes)
-		(effects
-			(font
-				(size 1.27 1.27)
-			)
-			(justify left)
-		)
-	)
-	(hierarchical_label "U+"
-		(shape input)
-		(at 86.36 74.93 90)
-		(fields_autoplaced yes)
-		(effects
-			(font
-				(size 1.27 1.27)
-			)
-			(justify left)
-		)
-	)
-	(hierarchical_label "AMP_MOTOR[0..1]"
-		(shape input)
-		(at 54.61 38.1 180)
 		(fields_autoplaced yes)
 		(effects
@@
 		(shape bidirectional)
 		(at 54.61 33.02 180)
-		(fields_autoplaced yes)
-		(effects
-			(font
-				(size 1.27 1.27)
-			)
-			(justify right)
-		)
-	)
-	(hierarchical_label "AUX[1..8]"
-		(shape input)
-		(at 54.61 49.53 180)
 		(fields_autoplaced yes)
 		(effects
@@
 		(dnp no)
 		(fields_autoplaced yes)
-		(property "Reference" "J106"
+		(property "Reference" "J301"
 			(at 55.88 71.12 0)
 			(effects
@@
 			(project "xDuinoRail-Debug"
 				(path "/3fe1c7d3-674a-46fe-b8de-0718a52fef91/ec041cac-ba8a-4e39-a1e2-0637cb1a7f49"
-					(reference "J106")
+					(reference "J301")
 					(unit 1)
 				)
@@
 		(dnp no)
 		(fields_autoplaced yes)
-		(property "Reference" "#PWR0103"
+		(property "Reference" "#PWR0301"
 			(at 92.71 93.98 0)
 			(effects
@@
 			(project "xDuinoRail-Debug"
 				(path "/3fe1c7d3-674a-46fe-b8de-0718a52fef91/ec041cac-ba8a-4e39-a1e2-0637cb1a7f49"
-					(reference "#PWR0103")
-					(unit 1)
-				)
+					(reference "#PWR0301")
+					(unit 1)
+				)

Commit message: More stuff
Parts:
- renumbered J301 to J5
Changed lines of the file:
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@@
 	(version 20231120)
 	(generator "eeschema")
-	(generator_version "7.99")
+	(generator_version "8.0")
 	(paper "A4")
 	(junction
@@
 		(dnp no)
 		(fields_autoplaced yes)
-		(property "Reference" "J301"
+		(property "Reference" "J5"
 			(at 55.88 71.12 0)
 			(effects
@@
 		)
 		(property "Description" "Generic connector, double row, 02x11, odd/even pin numbering scheme (row 1 odd numbers, row 2 even numbers), script generated (kicad-library-utils/schlib/autogen/connector/)"
+			(at 54.61 90.17 0)
+			(effects
+				(font
+					(size 1.27 1.27)
+				)
+				(hide yes)
+			)
+		)
+		(property "OLI_ID" ""
 			(at 54.61 90.17 0)
 			(effects
@@
 			(project "xDuinoRail-Debug"
 				(path "/3fe1c7d3-674a-46fe-b8de-0718a52fef91/ec041cac-ba8a-4e39-a1e2-0637cb1a7f49"
-					(reference "J301")
+					(reference "J5")
 					(unit 1)
 				)
@@
 		(dnp no)
 		(fields_autoplaced yes)
-		(property "Reference" "#PWR0301"
+		(property "Reference" "#PWR013"
 			(at 92.71 93.98 0)
 			(effects
@@
 			(project "xDuinoRail-Debug"
 				(path "/3fe1c7d3-674a-46fe-b8de-0718a52fef91/ec041cac-ba8a-4e39-a1e2-0637cb1a7f49"
-					(reference "#PWR0301")
+					(reference "#PWR013")
 					(unit 1)
 				)
