File: kicad/xDuinoRailShield/loco-adapter-nem651-6-pin.kicad_sch (KiCad schematic)
At the start: 7 parts, among them J104 Conn_01x06

Commit message: More refactoring
Parts:
- renumbered J104 to J401, JP102 to JP401, JP101 to JP402, JP104 to JP403, JP103 to JP404, JP105 to JP405, JP106 to JP406
Changed lines of the file:
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@@
 		(dnp yes)
 		(fields_autoplaced yes)
-		(property "Reference" "JP101"
+		(property "Reference" "JP402"
 			(at 52.07 86.36 0)
 			(effects
@@
 			(project "xDuinoRail-Debug"
 				(path "/3fe1c7d3-674a-46fe-b8de-0718a52fef91/a25ef325-35c0-450e-895f-b05e76b53aca"
-					(reference "JP101")
+					(reference "JP402")
 					(unit 1)
 				)
@@
 		(on_board yes)
 		(dnp yes)
-		(property "Reference" "JP103"
+		(property "Reference" "JP404"
 			(at 52.07 106.68 0)
 			(effects
@@
 			(project "xDuinoRail-Debug"
 				(path "/3fe1c7d3-674a-46fe-b8de-0718a52fef91/a25ef325-35c0-450e-895f-b05e76b53aca"
-					(reference "JP103")
+					(reference "JP404")
 					(unit 1)
 				)
@@
 		(dnp yes)
 		(fields_autoplaced yes)
-		(property "Reference" "JP106"
+		(property "Reference" "JP406"
 			(at 52.07 127 0)
 			(effects
@@
 			(project "xDuinoRail-Debug"
 				(path "/3fe1c7d3-674a-46fe-b8de-0718a52fef91/a25ef325-35c0-450e-895f-b05e76b53aca"
-					(reference "JP106")
+					(reference "JP406")
 					(unit 1)
 				)
@@
 		(dnp yes)
 		(fields_autoplaced yes)
-		(property "Reference" "JP104"
+		(property "Reference" "JP403"
 			(at 52.07 96.52 0)
 			(effects
@@
 			(project "xDuinoRail-Debug"
 				(path "/3fe1c7d3-674a-46fe-b8de-0718a52fef91/a25ef325-35c0-450e-895f-b05e76b53aca"
-					(reference "JP104")
+					(reference "JP403")
 					(unit 1)
 				)
@@
 		(dnp yes)
 		(fields_autoplaced yes)
-		(property "Reference" "JP105"
+		(property "Reference" "JP405"
 			(at 52.07 116.84 0)
 			(effects
@@
 			(project "xDuinoRail-Debug"
 				(path "/3fe1c7d3-674a-46fe-b8de-0718a52fef91/a25ef325-35c0-450e-895f-b05e76b53aca"
-					(reference "JP105")
+					(reference "JP405")
 					(unit 1)
 				)
@@
 		(on_board yes)
 		(dnp no)
-		(property "Reference" "J104"
+		(property "Reference" "J401"
 			(at 93.98 107.9499 0)
 			(effects
@@
 			(project "xDuinoRail-Debug"
 				(path "/3fe1c7d3-674a-46fe-b8de-0718a52fef91/a25ef325-35c0-450e-895f-b05e76b53aca"
-					(reference "J104")
+					(reference "J401")
 					(unit 1)
 				)
@@
 		(dnp yes)
 		(fields_autoplaced yes)
-		(property "Reference" "JP102"
+		(property "Reference" "JP401"
 			(at 52.07 76.2 0)
 			(effects
@@
 			(project "xDuinoRail-Debug"
 				(path "/3fe1c7d3-674a-46fe-b8de-0718a52fef91/a25ef325-35c0-450e-895f-b05e76b53aca"
-					(reference "JP102")
-					(unit 1)
-				)
+					(reference "JP401")
+					(unit 1)
+				)

Commit message: More stuff
Parts:
- renumbered J401 to J6, JP401 to JP1, JP402 to JP2, JP403 to JP3, JP404 to JP4, JP405 to JP5, JP406 to JP6
Changed lines of the file:
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@@
 	(version 20231120)
 	(generator "eeschema")
-	(generator_version "7.99")
+	(generator_version "8.0")
 	(paper "A4")
 	(no_connect
@@
 		(dnp yes)
 		(fields_autoplaced yes)
-		(property "Reference" "JP402"
+		(property "Reference" "JP2"
 			(at 52.07 86.36 0)
 			(effects
@@
 		)
 		(property "Description" "Solder Jumper, 2-pole, closed/bridged"
+			(at 52.07 92.71 0)
+			(effects
+				(font
+					(size 1.27 1.27)
+				)
+				(hide yes)
+			)
+		)
+		(property "OLI_ID" ""
 			(at 52.07 92.71 0)
 			(effects
@@
 			(project "xDuinoRail-Debug"
 				(path "/3fe1c7d3-674a-46fe-b8de-0718a52fef91/a25ef325-35c0-450e-895f-b05e76b53aca"
-					(reference "JP402")
+					(reference "JP2")
 					(unit 1)
 				)
@@
 		(on_board yes)
 		(dnp yes)
-		(property "Reference" "JP404"
+		(property "Reference" "JP4"
 			(at 52.07 106.68 0)
 			(effects
@@
 		)
 		(property "Description" "Solder Jumper, 2-pole, closed/bridged"
+			(at 52.07 113.03 0)
+			(effects
+				(font
+					(size 1.27 1.27)
+				)
+				(hide yes)
+			)
+		)
+		(property "OLI_ID" ""
 			(at 52.07 113.03 0)
 			(effects
@@
 			(project "xDuinoRail-Debug"
 				(path "/3fe1c7d3-674a-46fe-b8de-0718a52fef91/a25ef325-35c0-450e-895f-b05e76b53aca"
-					(reference "JP404")
+					(reference "JP4")
 					(unit 1)
 				)
@@
 		(dnp yes)
 		(fields_autoplaced yes)
-		(property "Reference" "JP406"
+		(property "Reference" "JP6"
 			(at 52.07 127 0)
 			(effects
@@
 		)
 		(property "Description" "Solder Jumper, 2-pole, closed/bridged"
+			(at 52.07 133.35 0)
+			(effects
+				(font
+					(size 1.27 1.27)
+				)
+				(hide yes)
+			)
+		)
+		(property "OLI_ID" ""
 			(at 52.07 133.35 0)
 			(effects
@@
 			(project "xDuinoRail-Debug"
 				(path "/3fe1c7d3-674a-46fe-b8de-0718a52fef91/a25ef325-35c0-450e-895f-b05e76b53aca"
-					(reference "JP406")
+					(reference "JP6")
 					(unit 1)
 				)
@@
 		(dnp yes)
 		(fields_autoplaced yes)
-		(property "Reference" "JP403"
+		(property "Reference" "JP3"
 			(at 52.07 96.52 0)
 			(effects
@@
 		)
 		(property "Description" "Solder Jumper, 2-pole, closed/bridged"
+			(at 52.07 102.87 0)
+			(effects
+				(font
+					(size 1.27 1.27)
+				)
+				(hide yes)
+			)
+		)
+		(property "OLI_ID" ""
 			(at 52.07 102.87 0)
 			(effects
@@
 			(project "xDuinoRail-Debug"
 				(path "/3fe1c7d3-674a-46fe-b8de-0718a52fef91/a25ef325-35c0-450e-895f-b05e76b53aca"
-					(reference "JP403")
+					(reference "JP3")
 					(unit 1)
 				)
@@
 		(dnp yes)
 		(fields_autoplaced yes)
-		(property "Reference" "JP405"
+		(property "Reference" "JP5"
 			(at 52.07 116.84 0)
 			(effects
@@
 		)
 		(property "Description" "Solder Jumper, 2-pole, closed/bridged"
+			(at 52.07 123.19 0)
+			(effects
+				(font
+					(size 1.27 1.27)
+				)
+				(hide yes)
+			)
+		)
+		(property "OLI_ID" ""
 			(at 52.07 123.19 0)
 			(effects
@@
 			(project "xDuinoRail-Debug"
 				(path "/3fe1c7d3-674a-46fe-b8de-0718a52fef91/a25ef325-35c0-450e-895f-b05e76b53aca"
-					(reference "JP405")
+					(reference "JP5")
 					(unit 1)
 				)
@@
 		(on_board yes)
 		(dnp no)
-		(property "Reference" "J401"
+		(property "Reference" "J6"
 			(at 93.98 107.9499 0)
 			(effects
@@
 		)
 		(property "Description" "Generic connector, single row, 01x06, script generated (kicad-library-utils/schlib/autogen/connector/)"
+			(at 91.44 107.95 0)
+			(effects
+				(font
+					(size 1.27 1.27)
+				)
+				(hide yes)
+			)
+		)
+		(property "OLI_ID" ""
 			(at 91.44 107.95 0)
 			(effects
@@
 			(project "xDuinoRail-Debug"
 				(path "/3fe1c7d3-674a-46fe-b8de-0718a52fef91/a25ef325-35c0-450e-895f-b05e76b53aca"
-					(reference "J401")
+					(reference "J6")
 					(unit 1)
 				)
@@
 		(dnp yes)
 		(fields_autoplaced yes)
-		(property "Reference" "JP401"
+		(property "Reference" "JP1"
 			(at 52.07 76.2 0)
 			(effects
@@
 		)
 		(property "Description" "Solder Jumper, 2-pole, closed/bridged"
+			(at 52.07 82.55 0)
+			(effects
+				(font
+					(size 1.27 1.27)
+				)
+				(hide yes)
+			)
+		)
+		(property "OLI_ID" ""
 			(at 52.07 82.55 0)
 			(effects
@@
 			(project "xDuinoRail-Debug"
 				(path "/3fe1c7d3-674a-46fe-b8de-0718a52fef91/a25ef325-35c0-450e-895f-b05e76b53aca"
-					(reference "JP401")
-					(unit 1)
-				)
+					(reference "JP1")
+					(unit 1)
+				)
