File: kicad/xDuinoRailShield/loco-adapter-nem652-8-pin.kicad_sch (KiCad schematic)
At the start: 1 part, among them J102 Conn_02x04_Counter_Clockwise

Commit message: More stuff
Parts:
- J1101: renamed from J102; footprint Connector_PinHeader_2.54mm:PinHeader_2x04_P2.54mm_Vertical_SMD -> Connector_PinHeader_2.54mm:PinHeader_2x04_P2.54mm_Vertical; now in the parts list
Changed lines of the file:
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@@
 	(version 20231120)
 	(generator "eeschema")
-	(generator_version "7.99")
+	(generator_version "8.0")
 	(paper "A4")
 	(no_connect
@@
 		(at 55.88 72.39 0)
 		(unit 1)
-		(exclude_from_sim yes)
-		(in_bom no)
-		(on_board no)
+		(exclude_from_sim no)
+		(in_bom yes)
+		(on_board yes)
 		(dnp yes)
 		(fields_autoplaced yes)
-		(property "Reference" "J102"
+		(property "Reference" "J1101"
 			(at 57.15 63.5 0)
 			(effects
@@
 			)
 		)
-		(property "Footprint" "Connector_PinHeader_2.54mm:PinHeader_2x04_P2.54mm_Vertical_SMD"
+		(property "Footprint" "Connector_PinHeader_2.54mm:PinHeader_2x04_P2.54mm_Vertical"
 			(at 55.88 72.39 0)
 			(effects
@@
 		)
 		(instances
+			(project "xDuinoRail-Debug"
+				(path "/3fe1c7d3-674a-46fe-b8de-0718a52fef91/f5a19207-1931-497e-ab27-14087bb9e856"
+					(reference "J1101")
+					(unit 1)
+				)
+			)
 			(project "loco-adapter-nem652-8-pin"
 				(path "/5e3bb3ff-c126-45cf-ab1e-9fd90e110c73"
-					(reference "J102")
+					(reference "J?")
 					(unit 1)
 				)
@@
 			(project "xDuinoRailShield"
 				(path "/e63e39d7-6ac0-4ffd-8aa3-1841a4541b55/a459cb8a-26f3-41b6-8de3-7368533e27fd"
-					(reference "J102")
+					(reference "J?")
 					(unit 1)
 				)
@@
 		)
 	)
-	(sheet_instances
-		(path "/"
-			(page "1")
-		)
-	)
