File: kicad/xDuinoRailShield/mcu_rp2040-onboard.kicad_sch (KiCad schematic)
At the start: 14 parts, among them J1001 SWCLK, J1002 SWDIO, J1003 RUN, J201 USB_B, U1003 RP2040, Y1001 X322512MSB4SI

Commit message: More stuff
Parts:
- removed J1001: SWCLK, TestPoint:TestPoint_Pad_D2.0mm, symbol Connector:Conn_01x01_Male
- removed J1002: SWDIO, TestPoint:TestPoint_Pad_D2.0mm, symbol Connector:Conn_01x01_Male
- removed J1003: RUN, TestPoint:TestPoint_Pad_D2.0mm, symbol Connector:Conn_01x01_Male
- added D1701: WS2812B, LED_SMD:LED_WS2812B_PLCC4_5.0x5.0mm_P3.2mm, symbol LED:WS2812B
- added R1703, R1704: 10k, Resistor_SMD:R_0805_2012Metric_Pad1.20x1.40mm_HandSolder, symbol Device:R
- C?: renamed from C1005; OLI_ID (none) -> 100nF_0805
- C?: renamed from C1006; OLI_ID (none) -> 10uF_0805
- C?: renamed from C1004; OLI_ID (none) -> 100nF_0805
- C?: renamed from C1012; OLI_ID (none) -> 10uF_0805
- J1701: renamed from J201; now not fitted
- R?: renamed from R1003; value 200R -> 220R; OLI_ID (none) -> 220R_0805
- R?: renamed from R1002; OLI_ID (none) -> 1k_0805
- U?: renamed from U1003; LCSC C2040 -> (none); OLI_ID (none) -> RP2040_LQFN-56
- Y?: renamed from Y1001; OLI_ID (none) -> X322512MSB4SI_SMD3225
- renumbered C1001 to C?, C1003 to C?
Connections:
- net +3V3: now also D1701.1 (VDD), R1703.1, R1704.1
- net GND: now also D1701.3 (VSS)
- net GPIO12: now also D1701.4 (DIN)
- net GPIO24: now also R1703.2
- net GPIO25: now also R1704.2
- net SWD: now reaches U?.25 (SWD)
- net USB_DM: now reaches J1701.2 (D-), U?.46 (USB_DM)
- net USB_DP: now reaches J1701.3 (D+), U?.47 (USB_DP)
- net TESTEN: now reaches U?.19 (TESTEN)
- net SWCLOCK: now reaches U?.24 (SWCLK)
- net RUN: now reaches U?.26 (RUN)
- no-connect marks 0 -> 1
Other:
- added sheet status-led (status-led.kicad_sch)
