File: kicad/xDuinoRailShield/rails_power_ac-dc-bridge-light.kicad_sch (KiCad schematic)
At the start: 4 parts

Commit message: More stuff
Parts:
- D?: renamed from D701; LCSC C191023 -> (none)
- D?: renamed from D702; LCSC C191023 -> (none)
- D?: renamed from D703; LCSC C191023 -> (none)
- D?: renamed from D704; LCSC C191023 -> (none)
Changed lines of the file:
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@@
 	(version 20231120)
 	(generator "eeschema")
-	(generator_version "7.99")
+	(generator_version "8.0")
 	(paper "A4")
 	(junction
@@
 		(on_board yes)
 		(dnp no)
-		(property "Reference" "D701"
+		(property "Reference" "D?"
 			(at 48.26 43.18 90)
 			(effects
@@
 		)
 		(property "Sim.Pins" "1=K 2=A"
-			(at 50.8 41.91 0)
-			(effects
-				(font
-					(size 1.27 1.27)
-				)
-				(hide yes)
-			)
-		)
-		(property "LCSC" "C191023"
 			(at 50.8 41.91 0)
 			(effects
@@
 			(project "power_ac-dc-bridge-light"
 				(path "/0ed6639a-cde6-4452-b9e1-77c370bade86"
-					(reference "D701")
+					(reference "D?")
+					(unit 1)
+				)
+			)
+			(project "xDuinoRail-Debug"
+				(path "/3fe1c7d3-674a-46fe-b8de-0718a52fef91/bf7aab3b-3930-4bc3-865d-386c1fe7edc1"
+					(reference "D1301")
 					(unit 1)
 				)
@@
 			(project "xDuinoRailSwitch"
 				(path "/e63e39d7-6ac0-4ffd-8aa3-1841a4541b55/36fdb63c-0a19-4659-9df1-d7f58d97597f"
-					(reference "D701")
+					(reference "D?")
 					(unit 1)
 				)
@@
 		(on_board yes)
 		(dnp no)
-		(property "Reference" "D702"
+		(property "Reference" "D?"
 			(at 55.88 31.75 0)
 			(effects
@@
 		)
 		(property "Sim.Pins" "1=K 2=A"
-			(at 55.88 38.1 0)
-			(effects
-				(font
-					(size 1.27 1.27)
-				)
-				(hide yes)
-			)
-		)
-		(property "LCSC" "C191023"
 			(at 55.88 38.1 0)
 			(effects
@@
 			(project "power_ac-dc-bridge-light"
 				(path "/0ed6639a-cde6-4452-b9e1-77c370bade86"
-					(reference "D702")
+					(reference "D?")
+					(unit 1)
+				)
+			)
+			(project "xDuinoRail-Debug"
+				(path "/3fe1c7d3-674a-46fe-b8de-0718a52fef91/bf7aab3b-3930-4bc3-865d-386c1fe7edc1"
+					(reference "D1302")
 					(unit 1)
 				)
@@
 			(project "xDuinoRailSwitch"
 				(path "/e63e39d7-6ac0-4ffd-8aa3-1841a4541b55/36fdb63c-0a19-4659-9df1-d7f58d97597f"
-					(reference "D702")
+					(reference "D?")
 					(unit 1)
 				)
@@
 		(on_board yes)
 		(dnp no)
-		(property "Reference" "D703"
+		(property "Reference" "D?"
 			(at 55.88 52.07 0)
 			(effects
@@
 		)
 		(property "Sim.Pins" "1=K 2=A"
-			(at 55.88 45.72 0)
-			(effects
-				(font
-					(size 1.27 1.27)
-				)
-				(hide yes)
-			)
-		)
-		(property "LCSC" "C191023"
 			(at 55.88 45.72 0)
 			(effects
@@
 			(project "power_ac-dc-bridge-light"
 				(path "/0ed6639a-cde6-4452-b9e1-77c370bade86"
-					(reference "D703")
+					(reference "D?")
+					(unit 1)
+				)
+			)
+			(project "xDuinoRail-Debug"
+				(path "/3fe1c7d3-674a-46fe-b8de-0718a52fef91/bf7aab3b-3930-4bc3-865d-386c1fe7edc1"
+					(reference "D1303")
 					(unit 1)
 				)
@@
 			(project "xDuinoRailSwitch"
 				(path "/e63e39d7-6ac0-4ffd-8aa3-1841a4541b55/36fdb63c-0a19-4659-9df1-d7f58d97597f"
-					(reference "D703")
+					(reference "D?")
 					(unit 1)
 				)
@@
 		(on_board yes)
 		(dnp no)
-		(property "Reference" "D704"
+		(property "Reference" "D?"
 			(at 62.23 43.18 90)
 			(effects
@@
 		)
 		(property "Sim.Pins" "1=K 2=A"
-			(at 59.69 41.91 0)
-			(effects
-				(font
-					(size 1.27 1.27)
-				)
-				(hide yes)
-			)
-		)
-		(property "LCSC" "C191023"
 			(at 59.69 41.91 0)
 			(effects
@@
 			(project "power_ac-dc-bridge-light"
 				(path "/0ed6639a-cde6-4452-b9e1-77c370bade86"
-					(reference "D704")
+					(reference "D?")
+					(unit 1)
+				)
+			)
+			(project "xDuinoRail-Debug"
+				(path "/3fe1c7d3-674a-46fe-b8de-0718a52fef91/bf7aab3b-3930-4bc3-865d-386c1fe7edc1"
+					(reference "D1304")
 					(unit 1)
 				)
@@
 			(project "xDuinoRailSwitch"
 				(path "/e63e39d7-6ac0-4ffd-8aa3-1841a4541b55/36fdb63c-0a19-4659-9df1-d7f58d97597f"
-					(reference "D704")
-					(unit 1)
-				)
-			)
-		)
-	)
-	(sheet_instances
-		(path "/"
-			(page "1")
-		)
-	)
+					(reference "D?")
+					(unit 1)
+				)
+			)
+		)
+	)
