File: kicad/xDuinoRailShield/rails_signal_feedback_dcc-railcom_BC8x7.kicad_sch (KiCad schematic)
At the start: 11 parts, among them Q901 BC847BVN, Q902 BC847BVN

Commit message: More stuff
Parts:
- removed R904, R905: 10k, Resistor_SMD:R_0805_2012Metric_Pad1.20x1.40mm_HandSolder, symbol Device:R
- removed TP901, TP902, TP903, TP904: TestPoint, TestPoint:TestPoint_Pad_D2.0mm, symbol Connector:TestPoint
- added D301: LED, LED_SMD:LED_0603_1608Metric_Pad1.05x0.95mm_HandSolder, symbol Device:LED
- added J301: Conn_01x05, Connector_PinHeader_2.54mm:PinHeader_1x05_P2.54mm_Vertical, symbol Connector_Generic:Conn_01x05
- added JP301: SolderJumper_2_Bridged, Jumper:SolderJumper-2_P1.3mm_Bridged_Pad1.0x1.5mm, symbol Jumper:SolderJumper_2_Bridged
- added R304, R305: 10k, Resistor_SMD:R_0805_2012Metric_Pad1.20x1.40mm_HandSolder, symbol Device:R
- added R306: 100R, Resistor_SMD:R_0805_2012Metric_Pad1.20x1.40mm_HandSolder, symbol Device:R
- Q301: renamed from Q901; OLI_ID (none) -> BC847BVN-7_SOT-563
- Q302: renamed from Q902; OLI_ID (none) -> BC847BVN-7_SOT-563
- R301: renamed from R901; LCSC C22950 -> (none)
- R302: renamed from R902; LCSC C22950 -> (none)
- R303: renamed from R903; LCSC C22950 -> (none)
Connections:
- net GND: now also D301.1 (K), J301.5 (Pin_5)
- net RAILCOM_DATA: now also J301.1 (Pin_1), JP301.2 (B), R305.2
- net RC_CURR: now also J301.2 (Pin_2)
- net RC_FB_IN: now also J301.3 (Pin_3), R305.1
- net RC_ON_OFF: now also J301.4 (Pin_4), R304.2
- net RC_SIGNAL: now also R304.1
- new net: D301.2 (A), R306.2
- new net: JP301.1 (A), R306.1
