File: kicad/xDuinoRailShield/xDuinoRailShield.kicad_pcb (KiCad board)
At the start: 2 copper layers, 59.7 x 21.9 mm, 19 parts, among them J105 21mtc_mrkl, Q501 S8050, Q502 S8550, Q503 S8550, Q504 S8050, U601 MOUDLE-SEEEDUINO-XIAO-ESP32C3, U801 L78L05_SOT89, U901 ULN2003A, U902 DRV8872DDA

Commit message: A lot of fixes
Parts:
- removed J105: 21mtc_mrkl, Connector_PinSocket_1.27mm:PinSocket_2x11_P1.27mm_Vertical_SMD
- added D503: LED, LED_SMD:LED_0805_2012Metric_Pad1.15x1.40mm_HandSolder, F.Cu at (162.2, 70.8)
- added J106: 21mtc_mrkl, Connector_PinSocket_1.27mm:PinSocket_2x11_P1.27mm_Vertical_SMD, F.Cu at (127.4, 74.6)
- added JP101: SolderJumper_2_Bridged, Jumper:SolderJumper-2_P1.3mm_Bridged_Pad1.0x1.5mm, B.Cu at (126.0, 70.8)
- added JP102: SolderJumper_2_Bridged, Jumper:SolderJumper-2_P1.3mm_Bridged_Pad1.0x1.5mm, B.Cu at (126.0, 68.2)
- added JP103: SolderJumper_2_Bridged, Jumper:SolderJumper-2_P1.3mm_Bridged_Pad1.0x1.5mm, B.Cu at (126.0, 75.9)
- added JP104: SolderJumper_2_Bridged, Jumper:SolderJumper-2_P1.3mm_Bridged_Pad1.0x1.5mm, B.Cu at (126.0, 73.3)
- added JP105: SolderJumper_2_Bridged, Jumper:SolderJumper-2_P1.3mm_Bridged_Pad1.0x1.5mm, B.Cu at (126.0, 78.4)
- added JP106: SolderJumper_2_Bridged, Jumper:SolderJumper-2_P1.3mm_Bridged_Pad1.0x1.5mm, B.Cu at (126.0, 81.0)
- added R503: 1k, Resistor_SMD:R_0805_2012Metric_Pad1.20x1.40mm_HandSolder, F.Cu at (157.2, 70.8)
- added U801: BDR6133, BDR6133:BDR6133, F.Cu at (153.3, 78.9)
- U902: value DRV8872DDA -> LIS3DH; footprint Package_SO:Texas_HTSOP-8-1EP_3.9x4.9mm_P1.27mm_EP2.95x4.9mm_Mask2.4x3.1mm_ThermalVias -> Package_LGA:LGA-16_3x3mm_P0.5mm_LayoutBorder3x5y
- moved R306 16.2 mm to (140.6, 72.1)
- moved U501 12.6 mm to (145.7, 85.4)
- moved R403 12.2 mm to (148.5, 80.8), turned to 90 degrees
- moved R401 10.7 mm to (147.0, 73.0), turned to 90 degrees
- moved D702 8.50 mm to (134.6, 72.9)
- moved U902 7.96 mm to (145.7, 82.2)
- moved U803 7.88 mm to (161.6, 77.4), turned to 90 degrees
- moved Q403 6.08 mm to (150.2, 72.1), turned to -90 degrees
- moved Q402 6.03 mm to (148.4, 77.0)
- moved R402 5.32 mm to (144.4, 73.1)
- moved Q404 4.58 mm to (144.8, 69.2)
- moved C705 3.27 mm to (145.0, 77.4), turned to -90 degrees
- moved D704 2.31 mm to (134.6, 76.7)
- moved U701 2.17 mm to (141.1, 79.0)
- moved Q401 1.84 mm to (140.9, 69.2)
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- renumbered C802 to C702, C805 to C705, D801 to D701, D802 to D702, D803 to D703, D804 to D704, Q501 to Q401, Q502 to Q402, Q503 to Q403, Q504 to Q404, R406 to R306, R501 to R401, R502 to R402, R503 to R403, U601 to U501, U801 to U701, U901 to U803
Connections:
- net /AUDIO renamed /MCU Carrier Board/EMF_MOTOR0
- net ACDC_SIGNAL renamed /MCU Carrier Board/EMF_MOTOR1
- net Net-(Q501-B) renamed /Railcom-Feedback/RC_SIGNAL
- net Net-(Q502-B) renamed /Railcom-Feedback/RC_FB_IN
- net Net-(Q502-E) renamed /Railcom-Feedback/RC_CURR
- net Net-(Q504-B) renamed /Railcom-Feedback/RC_ON_OFF
- U501 pad 12: unconnected-(U601-3V3-Pad12) -> +3V3
- U501 pad 6: /AUX2 -> /MCU Carrier Board/I2C1
- U501 pad 7: /AUX3 -> /MCU Carrier Board/I2C0
- U501 pad 8: /MCU Carrier Board/F0.BACKWARD -> /MCU Carrier Board/FUNC0
- U501 pad 9: /MCU Carrier Board/F0.FOREWARD -> /MCU Carrier Board/FUNC1
- U803 pad 1: /Motor and Power drivers/F00 -> /MCU Carrier Board/FUNC0
- U803 pad 10: /Motor and Power drivers/AMP_AUX5 -> unconnected-(U803-O7-Pad10)
- U803 pad 11: /Motor and Power drivers/AMP_AUX4 -> unconnected-(U803-O6-Pad11)
- U803 pad 12: AMP_AUX3 -> unconnected-(U803-O5-Pad12)
- U803 pad 13: AMP_AUX2 -> unconnected-(U803-O4-Pad13)
- U803 pad 14: AMP_AUX1 -> /Connectors 21mtc / PluXX / NEMA/AMP_AUX1
- U803 pad 15: /Motor and Power drivers/AMP_F01 -> /Connectors 21mtc / PluXX / NEMA/AMP_FUNC1
- U803 pad 16: /Motor and Power drivers/AMP_F00 -> /Connectors 21mtc / PluXX / NEMA/AMP_FUNC0
- U803 pad 2: /Motor and Power drivers/F01 -> /MCU Carrier Board/FUNC1
- U803 pad 4: /AUX2 -> unconnected-(U803-I4-Pad4)
- U803 pad 5: /AUX3 -> unconnected-(U803-I5-Pad5)
- U803 pad 6: /AUX4 -> unconnected-(U803-I6-Pad6)
- U803 pad 7: /AUX5 -> unconnected-(U803-I7-Pad7)
- U902 pad 1: GND -> +3V3
- U902 pad 2: /MCU Carrier Board/MOTOR1 -> unconnected-(U902-NC-Pad2)
- U902 pad 3: /MCU Carrier Board/MOTOR0 -> unconnected-(U902-NC-Pad3)
- U902 pad 4: unconnected-(U902-nFAULT-Pad4) -> /MCU Carrier Board/I2C0
- U902 pad 5: +5V -> GND
- U902 pad 6: /Connectors 21mtc / PluXX / NEMA/AMP_MOTOR0 -> /MCU Carrier Board/I2C1
- U902 pad 8: /Connectors 21mtc / PluXX / NEMA/AMP_MOTOR1 -> +3V3
- U902 pad 9: GND -> unconnected-(U902-INT2-Pad9)
Routing:
- net GND: track 114.0 -> 15.2 mm, vias 0 -> 13
- net AMP_AUX1: track 73.5 -> 0.00 mm
- net AMP_AUX3: track 66.7 -> 0.00 mm
- net /Connectors 21mtc / PluXX / NEMA/AMP_FUNC1: track 0.00 -> 63.3 mm, vias 0 -> 4
- net AMP_AUX2: track 54.9 -> 0.00 mm
- net /Connectors 21mtc / PluXX / NEMA/AMP_FUNC0: track 0.00 -> 39.3 mm, vias 0 -> 2
- net /Connectors 21mtc / PluXX / NEMA/AMP_AUX1: track 0.00 -> 35.2 mm, vias 0 -> 2
- net +3V3: track 0.00 -> 34.7 mm, vias 0 -> 5
- net DCC_VIN: track 18.5 -> 38.7 mm, vias 0 -> 2
- net /MCU Carrier Board/FUNC1: track 0.00 -> 19.4 mm
- net DCC_MM: track 41.8 -> 22.6 mm
- net RAILCOM_DATA: track 28.9 -> 9.74 mm, vias 1 -> 0
- net +5V: track 45.9 -> 64.4 mm, vias 1 -> 2
- net /Connectors 21mtc / PluXX / NEMA/AMP_MOTOR1: track 22.7 -> 38.7 mm
- net /MCU Carrier Board/FUNC0: track 0.00 -> 15.8 mm, vias 0 -> 1
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- added copper zone on B.Cu, net GND
Other:
- board size 59.7 x 21.9 mm -> 43.2 x 18.9 mm

Commit message: Final version
Parts:
- removed D503: LED, LED_SMD:LED_0805_2012Metric_Pad1.15x1.40mm_HandSolder
- removed R503: 1k, Resistor_SMD:R_0805_2012Metric_Pad1.20x1.40mm_HandSolder
- added JP401: J_EnableRailcom, Jumper:SolderJumper-2_P1.3mm_Bridged_RoundedPad1.0x1.5mm, B.Cu at (141.3, 74.6)
- added R801: 6K8, Resistor_SMD:R_0805_2012Metric_Pad1.20x1.40mm_HandSolder, F.Cu at (159.7, 82.2)
- added R802: 1K, Resistor_SMD:R_0805_2012Metric_Pad1.20x1.40mm_HandSolder, F.Cu at (164.8, 82.2)
- added R803: 6K8, Resistor_SMD:R_0805_2012Metric_Pad1.20x1.40mm_HandSolder, F.Cu at (159.4, 80.1)
- added R804: 1K, Resistor_SMD:R_0805_2012Metric_Pad1.20x1.40mm_HandSolder, F.Cu at (164.8, 80.2)
- moved C705 9.18 mm to (143.9, 68.2), turned to 180 degrees
- moved Q401 7.69 mm to (139.8, 76.8), turned to -90 degrees
- moved R306 7.68 mm to (140.1, 79.7)
- moved U701 6.77 mm to (140.7, 72.2)
- moved C702 6.39 mm to (139.9, 68.2)
- moved Q402 4.79 mm to (143.7, 77.6), turned to 90 degrees
- moved R401 4.19 mm to (147.5, 77.1), turned to 0 degrees
- moved D703 3.07 mm to (132.6, 78.2), turned to 90 degrees
- moved U803 2.62 mm to (161.7, 74.8)
- moved D702 2.59 mm to (136.2, 70.9), turned to -90 degrees
- moved D701 2.59 mm to (132.7, 70.7), turned to 90 degrees
- moved U801 2.46 mm to (153.6, 76.4)
- moved Q404 2.33 mm to (145.4, 71.5), turned to 90 degrees
- moved D704 2.29 mm to (136.3, 78.2), turned to -90 degrees
- moved R402 1.81 mm to (145.4, 74.6), turned to 0 degrees
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Connections:
- Q402 pad 3: /Railcom-Feedback/RC_SIGNAL -> Net-(JP401-A)
- R306 pad 1: /DCC0 -> /DCC1
- U803 pad 14: /Connectors 21mtc / PluXX / NEMA/AMP_AUX1 -> /Connectors 21mtc / PluXX / NEMA/AMP_FUNC1
- U803 pad 15: /Connectors 21mtc / PluXX / NEMA/AMP_FUNC1 -> /Connectors 21mtc / PluXX / NEMA/AMP_AUX1
- U803 pad 2: /MCU Carrier Board/FUNC1 -> /AUX1
- U803 pad 3: /AUX1 -> /MCU Carrier Board/FUNC1
Routing:
- net /Connectors 21mtc / PluXX / NEMA/AMP_FUNC1: track 63.3 -> 36.6 mm, vias 4 -> 2
- net /Connectors 21mtc / PluXX / NEMA/AMP_MOTOR1: track 38.7 -> 48.6 mm
- net /Railcom-Feedback/RC_SIGNAL: track 17.5 -> 7.66 mm, vias 3 -> 1
- net /MCU Carrier Board/EMF_MOTOR1: track 0.00 -> 8.73 mm
- net /DCC1: track 31.0 -> 38.6 mm, vias 2 -> 1
- net /MCU Carrier Board/I2C1: track 11.9 -> 4.97 mm, vias 1 -> 0
- net GND: track 15.2 -> 21.1 mm, vias 13 -> 9
- net Net-(D503-A): track 5.94 -> 0.00 mm
- net /MCU Carrier Board/FUNC1: track 19.4 -> 13.7 mm
- net /Connectors 21mtc / PluXX / NEMA/AMP_FUNC0: track 39.3 -> 33.8 mm
- net /MCU Carrier Board/EMF_MOTOR0: track 0.00 -> 5.47 mm
- net +5V: track 64.4 -> 59.2 mm, vias 2 -> 3
- net /Railcom-Feedback/RC_CURR: track 6.03 -> 10.5 mm
- net +3V3: track 34.7 -> 30.4 mm, vias 5 -> 2
- net Net-(JP401-A): track 0.00 -> 2.98 mm, vias 0 -> 1
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
Commit message: Refactoring & Sound
Parts:
- removed Q404: S8050, Package_TO_SOT_SMD:SOT-23
- removed U803: ULN2003A, Package_SO:SOIC-16_4.55x10.3mm_P1.27mm
- added Q801: 2N7002, Package_TO_SOT_SMD:SOT-23, F.Cu at (148.0, 71.4)
- added Q802: 2N7002, Package_TO_SOT_SMD:SOT-23, F.Cu at (134.0, 73.0)
- added Q803: 2N7002, Package_TO_SOT_SMD:SOT-23, F.Cu at (134.0, 69.5)
- added U201: MCP4725xxx-xCH, Package_TO_SOT_SMD:SOT-23-6_Handsoldering, F.Cu at (143.9, 80.5)
- C702, C705: footprint Capacitor_SMD:C_0805_2012Metric_Pad1.18x1.45mm_HandSolder -> Capacitor_SMD:C_0402_1005Metric_Pad0.74x0.62mm_HandSolder
- D701, D702, D703, D704: value SS34 -> 1N5819WS; footprint Diode_SMD:D_SMA -> Diode_SMD:D_SOD-323
- R306, R401, R402, R403, R801, R802, R803, R804: footprint Resistor_SMD:R_0805_2012Metric_Pad1.20x1.40mm_HandSolder -> Resistor_SMD:R_0402_1005Metric_Pad0.72x0.64mm_HandSolder
- moved R804 13.6 mm to (151.4, 82.9)
- moved U501 11.1 mm to (134.6, 85.4)
- moved Q402 11.0 mm to (153.0, 71.7)
- moved R802 10.8 mm to (154.0, 82.9), turned to 180 degrees
- moved U801 10.5 mm to (143.2, 74.6)
- moved C705 8.16 mm to (138.7, 74.6)
- moved R803 7.50 mm to (152.0, 81.0), turned to -90 degrees
- moved C702 7.27 mm to (136.4, 74.6)
- moved U701 6.65 mm to (137.6, 78.1)
- moved R403 6.53 mm to (154.6, 77.1)
- moved D702 6.19 mm to (133.7, 76.5), turned to 90 degrees
- moved D701 5.92 mm to (131.8, 76.5), turned to -90 degrees
- moved R401 5.51 mm to (150.8, 72.7), turned to -90 degrees
- moved R801 5.24 mm to (154.6, 81.0), turned to -90 degrees
- moved R402 5.15 mm to (150.2, 76.5), turned to -90 degrees
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Connections:
- net /Connectors 21mtc / PluXX / NEMA/SPEAKER1 renamed /Audio Interfaces/SPEAKER1
- net /MCU Carrier Board/I2C0 renamed /Audio Interfaces/I2C0
- net /MCU Carrier Board/I2C1 renamed /Audio Interfaces/I2C1
- net DCC_VIN renamed U+
- J106 pad 17: /Connectors 21mtc / PluXX / NEMA/SPEAKER0 -> /Audio Interfaces/SPEAKER0
- R306 pad 1: /DCC1 -> /DCC0
Routing:
- net /Audio Interfaces/SPEAKER0: track 0.00 -> 31.0 mm, vias 0 -> 2
- net /AUX1: track 10.8 -> 39.4 mm
- net /Connectors 21mtc / PluXX / NEMA/AMP_FUNC1: track 36.6 -> 9.17 mm
- net /Connectors 21mtc / PluXX / NEMA/AMP_AUX1: track 32.3 -> 4.93 mm, vias 2 -> 0
- net +5V: track 59.2 -> 45.8 mm, vias 3 -> 2
- net /DCC1: track 38.6 -> 28.0 mm, vias 1 -> 2
- net /Audio Interfaces/I2C0: track 3.72 -> 14.3 mm, vias 0 -> 2
- net DCC_MM: track 19.8 -> 11.0 mm, vias 0 -> 2
- net /Connectors 21mtc / PluXX / NEMA/AMP_MOTOR1: track 48.6 -> 39.9 mm
- net /Railcom-Feedback/RC_SIGNAL: track 7.66 -> 15.4 mm, vias 1 -> 2
- net Net-(JP401-A): track 2.98 -> 9.91 mm
- net /Railcom-Feedback/RC_CURR: track 10.5 -> 4.34 mm
- net /MCU Carrier Board/FUNC1: track 13.7 -> 7.79 mm
- net /Audio Interfaces/I2C1: track 4.97 -> 10.7 mm
- net /DCC0: track 36.2 -> 30.9 mm, vias 2 -> 1
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Other:
- board size 43.2 x 18.9 mm -> 31 x 19.1 mm

Commit message: More refactoring
Parts:
- removed R401: 20, Resistor_SMD:R_0402_1005Metric_Pad0.72x0.64mm_HandSolder
- added J104: Conn_01x06, Connector_Molex:Molex_KK-254_AE-6410-06A_1x06_P2.54mm_Vertical, F.Cu at (122.2, 81.0)
- added Q404: S8050, Package_TO_SOT_SMD:SOT-23, F.Cu at (149.2, 75.8)
- added R307: 10k, Resistor_SMD:R_0402_1005Metric_Pad0.72x0.64mm_HandSolder, F.Cu at (144.4, 79.0)
- added R404: 10R, Resistor_SMD:R_0402_1005Metric_Pad0.72x0.64mm_HandSolder, F.Cu at (150.8, 70.8)
- added R405: 10R, Resistor_SMD:R_0402_1005Metric_Pad0.72x0.64mm_HandSolder, F.Cu at (150.8, 72.1)
- added R406: 10R, Resistor_SMD:R_0402_1005Metric_Pad0.72x0.64mm_HandSolder, F.Cu at (150.8, 73.3)
- C705: footprint Capacitor_SMD:C_0402_1005Metric_Pad0.74x0.62mm_HandSolder -> Capacitor_SMD:C_0805_2012Metric_Pad1.18x1.45mm_HandSolder
- R306: value 22k -> 10k
- R402: value 6k8 -> 10k
- R801, R803: value 6K8 -> 10k
- U701: value L78L05_SOT89 -> HT7533-1
- moved JP102 12.8 mm to (128.0, 81.0), turned to 0 degrees
- moved JP106 12.8 mm to (128.0, 68.2), turned to 0 degrees
- moved JP401 11.5 mm to (152.1, 77.1)
- moved U201 7.98 mm to (138.0, 75.1)
- moved JP101 7.86 mm to (128.0, 78.4), turned to 0 degrees
- moved JP105 7.86 mm to (128.0, 70.8), turned to 0 degrees
- moved C705 7.38 mm to (142.7, 80.8), turned to 0 degrees
- moved C702 6.58 mm to (141.2, 79.0)
- moved Q802 4.42 mm to (133.2, 68.7)
- moved R402 3.87 mm to (146.4, 75.8)
- moved JP103 3.19 mm to (128.0, 73.3), turned to 0 degrees
- moved JP104 3.19 mm to (128.0, 75.9), turned to 0 degrees
- moved Q803 2.92 mm to (133.4, 72.4), turned to 0 degrees
- moved R306 2.92 mm to (135.8, 82.6)
- moved R403 2.24 mm to (153.4, 79.0), turned to 180 degrees
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Connections:
- C705 pad 1: +5V -> +3V3
- J106 pad 22: +5V -> /Connectors 21mtc / PluXX / NEMA/+3V3
- JP101 pad 2: /DCC0 -> /Connectors 21mtc / PluXX / NEMA/AMP_MOTOR0
- JP102 pad 2: /DCC1 -> /Connectors 21mtc / PluXX / NEMA/AMP_MOTOR1
- JP103 pad 2: /Connectors 21mtc / PluXX / NEMA/AMP_MOTOR0 -> /DCC0
- JP104 pad 2: /Connectors 21mtc / PluXX / NEMA/AMP_MOTOR1 -> /DCC1
- JP105 pad 2: /Connectors 21mtc / PluXX / NEMA/FUNC0 -> /Connectors 21mtc / PluXX / NEMA/FUNC1
- JP106 pad 2: /Connectors 21mtc / PluXX / NEMA/FUNC1 -> /Connectors 21mtc / PluXX / NEMA/FUNC0
- Q403 pad 1: +5V -> +3V3
- R306 pad 1: /DCC0 -> /DCC1
- R306 pad 2: DCC_MM -> Net-(R306-Pad2)
- U201 pad 1: /Audio Interfaces/SPEAKER0 -> /Audio Interfaces/SPEAKER1
- U701 pad 1: +5V -> +3V3
- U801 pad 2: +5V -> +3V3
Routing:
- net +5V: track 45.8 -> 0.00 mm, vias 2 -> 0
- net /Audio Interfaces/SPEAKER0: track 31.0 -> 0.00 mm, vias 2 -> 0
- net /AUX1: track 39.4 -> 18.7 mm
- net U+: track 42.4 -> 22.1 mm
- net /Connectors 21mtc / PluXX / NEMA/AMP_MOTOR1: track 39.9 -> 59.6 mm
- net /Audio Interfaces/SPEAKER1: track 0.00 -> 17.6 mm, vias 0 -> 2
- net +3V3: track 26.0 -> 9.27 mm, vias 1 -> 9
- net /DCC0: track 30.9 -> 42.1 mm, vias 1 -> 2
- net Net-(R306-Pad2): track 0.00 -> 9.65 mm
- net /Connectors 21mtc / PluXX / NEMA/FUNC1: track 0.00 -> 8.60 mm
- net /Connectors 21mtc / PluXX / NEMA/FUNC0: track 0.00 -> 7.83 mm
- net /Audio Interfaces/I2C1: track 10.7 -> 17.8 mm, vias 0 -> 1
- net /Audio Interfaces/I2C0: track 14.3 -> 19.9 mm
- net /MCU Carrier Board/EMF_MOTOR1: track 3.78 -> 9.34 mm, vias 0 -> 1
- net DCC_MM: track 11.0 -> 6.62 mm, vias 2 -> 1
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- added copper zone on In2.Cu, net +3V3
- added copper zone on In1.Cu, net GND
- removed copper zone on B.Cu, net GND
Other:
- board size 31 x 19.1 mm -> 34.3 x 19.7 mm
- copper layers 2 -> 4
