File: kicad/xDuinoRailShield/centrale-driver-8874.kicad_sch (KiCad schematic)
At the start: 12 parts, among them U4 DRV8874PWPR

Commit message: Neue Breakouts
Parts:
- removed D2901: LED_RED, LED_SMD:LED_0603_1608Metric_Pad1.05x0.95mm_HandSolder, symbol Device:LED
- removed D2902: LED_YELLOW, LED_SMD:LED_0603_1608Metric_Pad1.05x0.95mm_HandSolder, symbol Device:LED
- removed D2903: LED_GREEN, LED_SMD:LED_0603_1608Metric_Pad1.05x0.95mm_HandSolder, symbol Device:LED
- removed R2901, R2902, R2903: 470R, Resistor_SMD:R_0805_2012Metric_Pad1.20x1.40mm_HandSolder, symbol Device:R
- C3, C5: OLI_ID (none) -> 22nF_0805
- C4: OLI_ID (none) -> 100nF_0805
- R2: OLI_ID (none) -> 47k_0805
- R3: value 1k5 -> 1k; OLI_ID (none) -> 1k_0805
Other:
- moved on the sheet: R2
