File: kicad/xDuinoRailShield/xDuinoRail-Breakout-DRV8874.kicad_sch (KiCad schematic)
At the start: 1 part, among them J101 Conn_01x09

Commit message: Neue Breakouts
Parts:
- removed J101: Conn_01x09, Connector_PinHeader_2.54mm:PinHeader_1x09_P2.54mm_Horizontal, symbol Connector_Generic:Conn_01x09
- added D101: LED_RED, LED_SMD:LED_0603_1608Metric_Pad1.05x0.95mm_HandSolder, symbol Device:LED
- added D102: LED_YELLOW, LED_SMD:LED_0603_1608Metric_Pad1.05x0.95mm_HandSolder, symbol Device:LED
- added D103: LED_GREEN, LED_SMD:LED_0603_1608Metric_Pad1.05x0.95mm_HandSolder, symbol Device:LED
- added J101: Conn_02x06_Odd_Even, Connector_PinHeader_2.54mm:PinHeader_2x06_P2.54mm_Horizontal, symbol Connector_Generic:Conn_02x06_Odd_Even
- added R101, R102, R103: 470R, Resistor_SMD:R_0805_2012Metric_Pad1.20x1.40mm_HandSolder, symbol Device:R
Connections:
- net +3V3: now also J101.5 (Pin_5)
- net +VIN: now also J101.9 (Pin_9)
- net DCC0: now also J101.1 (Pin_1)
- net DCC1: now also J101.3 (Pin_3)
- net GND: now also D101.1 (K), D102.1 (K), D103.1 (K), J101.7 (Pin_7)
- net centrale-driver-8874/SENSE: now also J101.12 (Pin_12)
- new net: D101.2 (A), R101.2
- new net: D102.2 (A), R102.2
- new net: D103.2 (A), R103.2
- new net BRAKE: J101.6 (Pin_6), R101.1
- new net DIR: J101.8 (Pin_8), R102.1
- new net PWM: J101.10 (Pin_10), R103.1
- no-connect marks 0 -> 3
