File: kicad/xDuinoRailShield/central_railcom-detector.kicad_sch (KiCad schematic)
At the start: 20 parts, among them U103 LM339

Commit message: More refactoring
Parts:
- removed D105: 1N5400, Diode_THT:D_DO-201AD_P15.24mm_Horizontal, symbol Diode:1N5400
- removed unit 1 of U103
- removed unit 2 of U103
- added D505: SS54, Diode_SMD:D_SMA-SMB_Universal_Handsoldering, symbol Device:D
- added unit 2 of U501
- added unit 1 of U501
- C501: renamed from C101; footprint (none) -> Capacitor_SMD:C_0805_2012Metric_Pad1.18x1.45mm_HandSolder
- D503: renamed from D101; value 1N5400 -> SS54; footprint Diode_THT:D_DO-201AD_P15.24mm_Horizontal -> Diode_SMD:D_SMA-SMB_Universal_Handsoldering
- D504: renamed from D102; value 1N5400 -> SS54; footprint Diode_THT:D_DO-201AD_P15.24mm_Horizontal -> Diode_SMD:D_SMA-SMB_Universal_Handsoldering
- D506: renamed from D106; value 1N5400 -> SS54; footprint Diode_THT:D_DO-201AD_P15.24mm_Horizontal -> Diode_SMD:D_SMA-SMB_Universal_Handsoldering
- renumbered D103 to D501, D104 to D502, R108 to R501, R109 to R502, R103 to R503, R102 to R504, R106 to R505, R107 to R506, R110 to R507, R101 to R508, R111 to R509, R112 to R510, R104 to R511, R105 to R512, U103 to U501
Connections:
- net +18mV: now also U501.7 (+)
- net -18mv: now also U501.4 (-)
- net DCC_CTRL0: now also D505.1 (K)
- net DCC_TRACK_A0: now also U501.5 (+), U501.6 (-)
- net DCC_TRACK_B0: now also D505.2 (A)
- net RAILCOM_A1: now reaches R509.1
- net RAILCOM_A1: now also U501.1
- net RAILCOM_A0: now reaches R510.1
- net RAILCOM_A0: now also U501.2
- net RAILCOM_B1: now reaches R511.1, U501.14
- net RAILCOM_B0: now reaches R512.1, U501.13

Commit message: More stuff
Parts:
- removed C501: 47uF, Capacitor_SMD:C_0805_2012Metric_Pad1.18x1.45mm_HandSolder, symbol Device:C_Polarized
- removed D501, D502: 1N4004, Diode_SMD:D_SOD-123F, symbol Diode:1N4004
- removed D503, D504, D506: SS54, Diode_SMD:D_SMA-SMB_Universal_Handsoldering, symbol Diode:1N5400
- removed D505: SS54, Diode_SMD:D_SMA-SMB_Universal_Handsoldering, symbol Device:D
- removed R501, R502: 220R, Resistor_SMD:R_0805_2012Metric_Pad1.20x1.40mm_HandSolder, symbol Device:R
- removed R503: 270K, Resistor_SMD:R_0805_2012Metric_Pad1.20x1.40mm_HandSolder, symbol Device:R
- removed R504: 1K, Resistor_SMD:R_0805_2012Metric_Pad1.20x1.40mm_HandSolder, symbol Device:R
- removed R505: 820R, Resistor_SMD:R_0805_2012Metric_Pad1.20x1.40mm_HandSolder, symbol Device:R
- removed R506: 33k, Resistor_SMD:R_0805_2012Metric_Pad1.20x1.40mm_HandSolder, symbol Device:R
- removed unit 5 of U501
- added D2401, D2402, D2403, D2404: SS54, Diode_SMD:D_SMA-SMB_Universal_Handsoldering, symbol Device:D
- added unit 5 of U2401
- R2401: renamed from R507; OLI_ID (none) -> 1R8_0805
- R2402: renamed from R508; OLI_ID (none) -> 1R8_0805
- R2403: renamed from R509; value 10K -> 10k; OLI_ID (none) -> 10k_0805
- R2404: renamed from R510; value 10K -> 10k; OLI_ID (none) -> 10k_0805
- R2405: renamed from R511; value 10K -> 10k; OLI_ID (none) -> 10k_0805
- R2406: renamed from R512; value 10K -> 10k; OLI_ID (none) -> 10k_0805
- U2401: renamed from U501; OLI_ID (none) -> LM339_SOIC-14
Connections:
- net DCC_CTRL0: now also D2401.1 (K), D2402.2 (A), D2403.1 (K), D2404.2 (A)
- net DCC_TRACK_A0: now also D2401.2 (A), D2402.1 (K)
- net DCC_TRACK_B0: now also D2403.2 (A), D2404.1 (K)
- net +5V renamed +3V3
- net +3V3: now also U2401.3 (V+)
- net -18mv renamed -18mV
- new net -750mV: U2401.12 (V-)
Other:
- note removed: "3V3 / 180 = 18mV"
- note removed: "5V / 270 = 18mV"
- note removed: "Forward voltage of 1N4004 at 30mA"
- moved on the sheet: R2401, R2402, R2403, R2404, R2405, R2406, U2401A, U2401B, U2401C, U2401D

Commit message: Many exiting news
Parts:
- added RN501: R_Pack04_SIP_Split, Resistor_SMD:R_Array_Convex_4x0603, symbol Device:R_Pack04_SIP_Split
- D501: renamed from D2401; footprint Diode_SMD:D_SMA-SMB_Universal_Handsoldering -> Diode_SMD:D_SMA_Handsoldering
- D502: renamed from D2402; footprint Diode_SMD:D_SMA-SMB_Universal_Handsoldering -> Diode_SMD:D_SMA_Handsoldering
- D503: renamed from D2403; footprint Diode_SMD:D_SMA-SMB_Universal_Handsoldering -> Diode_SMD:D_SMA_Handsoldering
- D504: renamed from D2404; footprint Diode_SMD:D_SMA-SMB_Universal_Handsoldering -> Diode_SMD:D_SMA_Handsoldering
- R501: renamed from R2401; value 1R8 -> 2R; OLI_ID 1R8_0805 -> 2R_0603
- R502: renamed from R2402; value 1R8 -> 2R; OLI_ID 1R8_0805 -> 2R_0603
- renumbered R2403 to R503, R2404 to R504, R2405 to R505, R2406 to R506, U2401 to U501
Connections:
- net +3V3: now also RN501.2 (R1.2), RN501.4 (R2.2), RN501.6 (R3.2), RN501.8 (R4.2)
- net RAILCOM_A0: now also RN501.3 (R2.1)
- net RAILCOM_A1: now also RN501.1 (R1.1)
- net RAILCOM_B0: now also RN501.7 (R4.1)
- net RAILCOM_B1: now also RN501.5 (R3.1)
