File: kicad/xDuinoRailShield/central_railcom-merger.kicad_sch (KiCad schematic)
At the start: 1 part, among them U2501 74HC02

Commit message: Many exiting news
Parts:
- added C601: 100uF, Capacitor_SMD:C_1206_3216Metric_Pad1.33x1.80mm_HandSolder, symbol Device:C
- added C602: 100nF, Capacitor_SMD:C_0805_2012Metric_Pad1.18x1.45mm_HandSolder, symbol Device:C
- U601: renamed from U2501; footprint Package_SO:SOIC-14-16_3.9x9.9mm_P1.27mm -> Package_SO:SOIC-14_3.9x8.7mm_P1.27mm
Connections:
- net +3V3: now also C601.1, C602.1
- net GND: now also C601.2, C602.2
Other:
- moved on the sheet: U601A
