File: kicad/xDuinoRailShield/central_railcom-power-source.kicad_sch (KiCad schematic)
At the start: 9 parts

Commit message: Many exiting news
Parts:
- removed C2301: 47uF, Capacitor_SMD:C_0805_2012Metric_Pad1.18x1.45mm_HandSolder, symbol Device:C_Polarized
- removed D2301, D2302: SM4007, Diode_SMD:D_SMA-SMB_Universal_Handsoldering, symbol Diode:SM4007
- removed R2301, R2302: 220R, Resistor_SMD:R_0805_2012Metric_Pad1.20x1.40mm_HandSolder, symbol Device:R
- added C401: 47uF, Capacitor_SMD:C_0805_2012Metric_Pad1.18x1.45mm_HandSolder, symbol Device:C_Polarized
- added D401, D402: SM4007, Diode_SMD:D_SMA_Handsoldering, symbol Diode:SM4007
- added R401, R402, R406: 220R, Resistor_SMD:R_0805_2012Metric_Pad1.20x1.40mm_HandSolder, symbol Device:R
- added R405: 10k, Resistor_SMD:R_0805_2012Metric_Pad1.20x1.40mm_HandSolder, symbol Device:R
- R403: renamed from R2304; value 1k -> 220R; OLI_ID 1k_0805 -> 220R_0805
- R404: renamed from R2303; value 180K -> 10k; OLI_ID 220k_0805 -> 10k_0805
- R407: renamed from R2305; value 820R -> 220R; OLI_ID 820R_0805 -> 220R_0805
- R408: renamed from R2306; value 33k -> 10k; OLI_ID 33k_0805 -> 10k_0805
Connections:
- net +18mV: now also R405.1, R406.2; no longer R404.1
- net -750mV: now also D402.1 (K), R402.1
- net GND: now also C401.1, D402.2 (A), R406.1
- new net: D401.2 (A), R401.2
- new net: R404.1, R405.2
- new net DCC_CTRL1: D401.1 (K)
- new net DCC_NEG: C401.2, R401.1, R402.2
Other:
- note added: "Forward voltage 1N4004: - 750mV at 30mA - 1'000mV at 1'000MA"
- note added: "RCN-217: 5v with 1k : 270k = +18mV xDuinoRail: 3v3 with 1k : 200k = +16mV"
- note added: "RCN-217: 750 with 820R : 33k = -18mV xDuinoRail: 750 with 220R : 10k = -16mV"
- note removed: "3V3 / 180 = 18mV"
- note removed: "5V / 270 = 18mV"
- moved on the sheet: R403, R404, R407, R408
