File: kicad/xDuinoRailShield/loco-track-terminal.kicad_sch (KiCad schematic)
At the start: 5 parts, among them J601 Screw_Terminal_01x02

Commit message: More stuff
Parts:
- D2801: renamed from D601; footprint LED_SMD:LED_0805_2012Metric_Pad1.15x1.40mm_HandSolder -> LED_SMD:LED_0603_1608Metric_Pad1.05x0.95mm_HandSolder; LCSC C2297 -> (none); OLI_ID (none) -> LED-RED_0603
- D2802: renamed from D602; footprint LED_SMD:LED_0805_2012Metric_Pad1.15x1.40mm_HandSolder -> LED_SMD:LED_0603_1608Metric_Pad1.05x0.95mm_HandSolder; LCSC C2297 -> (none); OLI_ID (none) -> LED-RED_0603
- J2801: renamed from J601; LCSC C8269 -> (none); OLI_ID (none) -> Spring_Terminal_01x02
- R2801: renamed from R601; LCSC C26010 -> (none); OLI_ID (none) -> 3k3_0805
- R2802: renamed from R602; LCSC C26010 -> (none); OLI_ID (none) -> 3k3_0805
Changed lines of the file:
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@@
 	(version 20231120)
 	(generator "eeschema")
-	(generator_version "7.99")
+	(generator_version "8.0")
 	(paper "A4")
 	(junction
@@
 		(on_board yes)
 		(dnp no)
-		(property "Reference" "J601"
+		(property "Reference" "J2801"
 			(at 72.39 44.45 0)
 			(effects
@@
 			)
 		)
-		(property "LCSC" "C8269"
-			(at 72.39 41.91 0)
-			(effects
-				(font
-					(size 1.27 1.27)
-				)
-				(hide yes)
-			)
-		)
 		(property "Field-1" ""
 			(at 72.39 41.91 0)
@@
 			)
 		)
+		(property "OLI_ID" "Spring_Terminal_01x02"
+			(at 72.39 41.91 0)
+			(effects
+				(font
+					(size 1.27 1.27)
+				)
+				(hide yes)
+			)
+		)
 		(pin "1"
 		)
@@
 		(instances
 			(project "xDuinoRail-Debug"
-				(path "/3fe1c7d3-674a-46fe-b8de-0718a52fef91/e428b020-e8a0-4fd3-b33d-3831684b9770"
-					(reference "J601")
-					(unit 1)
-				)
-				(path "/3fe1c7d3-674a-46fe-b8de-0718a52fef91/379ceeb1-29cb-43d0-b953-00e5101be218"
-					(reference "J801")
-					(unit 1)
-				)
-				(path "/3fe1c7d3-674a-46fe-b8de-0718a52fef91/869ab187-d4c3-4427-843d-f3d1f0f0aa48"
-					(reference "J701")
+				(path "/3fe1c7d3-674a-46fe-b8de-0718a52fef91/a69e15f3-9c14-4aca-9191-41e586ada203/b77f0077-1926-4790-a8ae-2d9cb2a861f8"
+					(reference "J2801")
+					(unit 1)
+				)
+				(path "/3fe1c7d3-674a-46fe-b8de-0718a52fef91/a69e15f3-9c14-4aca-9191-41e586ada203/3b3a13db-6557-433d-96a5-218459e8b091"
+					(reference "J2601")
+					(unit 1)
+				)
+				(path "/3fe1c7d3-674a-46fe-b8de-0718a52fef91/a69e15f3-9c14-4aca-9191-41e586ada203/cbcba9a5-81e5-4be6-bbd1-91127981b75d"
+					(reference "J2701")
 					(unit 1)
 				)
@@
 		(on_board yes)
 		(dnp no)
-		(property "Reference" "D601"
+		(property "Reference" "D2801"
 			(at 30.48 45.4025 90)
 			(effects
@@
 			)
 		)
-		(property "Footprint" "LED_SMD:LED_0805_2012Metric_Pad1.15x1.40mm_HandSolder"
+		(property "Footprint" "LED_SMD:LED_0603_1608Metric_Pad1.05x0.95mm_HandSolder"
 			(at 34.29 45.72 0)
 			(effects
@@
 			)
 		)
-		(property "LCSC" "C2297"
-			(at 34.29 45.72 0)
-			(effects
-				(font
-					(size 1.27 1.27)
-				)
-				(hide yes)
-			)
-		)
 		(property "Field-1" ""
 			(at 34.29 45.72 0)
@@
 			)
 		)
+		(property "OLI_ID" "LED-RED_0603"
+			(at 34.29 45.72 0)
+			(effects
+				(font
+					(size 1.27 1.27)
+				)
+				(hide yes)
+			)
+		)
 		(pin "1"
 		)
@@
 		(instances
 			(project "xDuinoRail-Debug"
-				(path "/3fe1c7d3-674a-46fe-b8de-0718a52fef91/e428b020-e8a0-4fd3-b33d-3831684b9770"
-					(reference "D601")
-					(unit 1)
-				)
-				(path "/3fe1c7d3-674a-46fe-b8de-0718a52fef91/379ceeb1-29cb-43d0-b953-00e5101be218"
-					(reference "D801")
-					(unit 1)
-				)
-				(path "/3fe1c7d3-674a-46fe-b8de-0718a52fef91/869ab187-d4c3-4427-843d-f3d1f0f0aa48"
-					(reference "D701")
+				(path "/3fe1c7d3-674a-46fe-b8de-0718a52fef91/a69e15f3-9c14-4aca-9191-41e586ada203/b77f0077-1926-4790-a8ae-2d9cb2a861f8"
+					(reference "D2801")
+					(unit 1)
+				)
+				(path "/3fe1c7d3-674a-46fe-b8de-0718a52fef91/a69e15f3-9c14-4aca-9191-41e586ada203/3b3a13db-6557-433d-96a5-218459e8b091"
+					(reference "D2601")
+					(unit 1)
+				)
+				(path "/3fe1c7d3-674a-46fe-b8de-0718a52fef91/a69e15f3-9c14-4aca-9191-41e586ada203/cbcba9a5-81e5-4be6-bbd1-91127981b75d"
+					(reference "D2701")
 					(unit 1)
 				)
@@
 		(on_board yes)
 		(dnp no)
-		(property "Reference" "R602"
+		(property "Reference" "R2802"
 			(at 44.45 43.18 0)
 			(effects
@@
 			)
 		)
-		(property "LCSC" "C26010"
-			(at 41.91 44.45 0)
-			(effects
-				(font
-					(size 1.27 1.27)
-				)
-				(hide yes)
-			)
-		)
 		(property "Field-1" ""
 			(at 41.91 44.45 0)
@@
 			)
 		)
+		(property "OLI_ID" "3k3_0805"
+			(at 41.91 44.45 0)
+			(effects
+				(font
+					(size 1.27 1.27)
+				)
+				(hide yes)
+			)
+		)
 		(pin "1"
 		)
@@
 		(instances
 			(project "xDuinoRail-Debug"
-				(path "/3fe1c7d3-674a-46fe-b8de-0718a52fef91/e428b020-e8a0-4fd3-b33d-3831684b9770"
-					(reference "R602")
-					(unit 1)
-				)
-				(path "/3fe1c7d3-674a-46fe-b8de-0718a52fef91/379ceeb1-29cb-43d0-b953-00e5101be218"
-					(reference "R802")
-					(unit 1)
-				)
-				(path "/3fe1c7d3-674a-46fe-b8de-0718a52fef91/869ab187-d4c3-4427-843d-f3d1f0f0aa48"
-					(reference "R702")
+				(path "/3fe1c7d3-674a-46fe-b8de-0718a52fef91/a69e15f3-9c14-4aca-9191-41e586ada203/b77f0077-1926-4790-a8ae-2d9cb2a861f8"
+					(reference "R2802")
+					(unit 1)
+				)
+				(path "/3fe1c7d3-674a-46fe-b8de-0718a52fef91/a69e15f3-9c14-4aca-9191-41e586ada203/3b3a13db-6557-433d-96a5-218459e8b091"
+					(reference "R2602")
+					(unit 1)
+				)
+				(path "/3fe1c7d3-674a-46fe-b8de-0718a52fef91/a69e15f3-9c14-4aca-9191-41e586ada203/cbcba9a5-81e5-4be6-bbd1-91127981b75d"
+					(reference "R2702")
 					(unit 1)
 				)
@@
 		(on_board yes)
 		(dnp no)
-		(property "Reference" "R601"
+		(property "Reference" "R2801"
 			(at 31.75 54.61 0)
 			(effects
@@
 			)
 		)
-		(property "LCSC" "C26010"
-			(at 34.29 53.34 0)
-			(effects
-				(font
-					(size 1.27 1.27)
-				)
-				(hide yes)
-			)
-		)
 		(property "Field-1" ""
 			(at 34.29 53.34 0)
@@
 			)
 		)
+		(property "OLI_ID" "3k3_0805"
+			(at 34.29 53.34 0)
+			(effects
+				(font
+					(size 1.27 1.27)
+				)
+				(hide yes)
+			)
+		)
 		(pin "1"
 		)
@@
 		(instances
 			(project "xDuinoRail-Debug"
-				(path "/3fe1c7d3-674a-46fe-b8de-0718a52fef91/e428b020-e8a0-4fd3-b33d-3831684b9770"
-					(reference "R601")
-					(unit 1)
-				)
-				(path "/3fe1c7d3-674a-46fe-b8de-0718a52fef91/379ceeb1-29cb-43d0-b953-00e5101be218"
-					(reference "R801")
-					(unit 1)
-				)
-				(path "/3fe1c7d3-674a-46fe-b8de-0718a52fef91/869ab187-d4c3-4427-843d-f3d1f0f0aa48"
-					(reference "R701")
+				(path "/3fe1c7d3-674a-46fe-b8de-0718a52fef91/a69e15f3-9c14-4aca-9191-41e586ada203/b77f0077-1926-4790-a8ae-2d9cb2a861f8"
+					(reference "R2801")
+					(unit 1)
+				)
+				(path "/3fe1c7d3-674a-46fe-b8de-0718a52fef91/a69e15f3-9c14-4aca-9191-41e586ada203/3b3a13db-6557-433d-96a5-218459e8b091"
+					(reference "R2601")
+					(unit 1)
+				)
+				(path "/3fe1c7d3-674a-46fe-b8de-0718a52fef91/a69e15f3-9c14-4aca-9191-41e586ada203/cbcba9a5-81e5-4be6-bbd1-91127981b75d"
+					(reference "R2701")
 					(unit 1)
 				)
@@
 		(on_board yes)
 		(dnp no)
-		(property "Reference" "D602"
+		(property "Reference" "D2802"
 			(at 45.72 52.3875 90)
 			(effects
@@
 			)
 		)
-		(property "Footprint" "LED_SMD:LED_0805_2012Metric_Pad1.15x1.40mm_HandSolder"
+		(property "Footprint" "LED_SMD:LED_0603_1608Metric_Pad1.05x0.95mm_HandSolder"
 			(at 41.91 52.07 0)
 			(effects
@@
 			)
 		)
-		(property "LCSC" "C2297"
-			(at 41.91 52.07 0)
-			(effects
-				(font
-					(size 1.27 1.27)
-				)
-				(hide yes)
-			)
-		)
 		(property "Field-1" ""
 			(at 41.91 52.07 0)
@@
 			)
 		)
+		(property "OLI_ID" "LED-RED_0603"
+			(at 41.91 52.07 0)
+			(effects
+				(font
+					(size 1.27 1.27)
+				)
+				(hide yes)
+			)
+		)
 		(pin "1"
 		)
@@
 		(instances
 			(project "xDuinoRail-Debug"
-				(path "/3fe1c7d3-674a-46fe-b8de-0718a52fef91/e428b020-e8a0-4fd3-b33d-3831684b9770"
-					(reference "D602")
-					(unit 1)
-				)
-				(path "/3fe1c7d3-674a-46fe-b8de-0718a52fef91/379ceeb1-29cb-43d0-b953-00e5101be218"
-					(reference "D802")
-					(unit 1)
-				)
-				(path "/3fe1c7d3-674a-46fe-b8de-0718a52fef91/869ab187-d4c3-4427-843d-f3d1f0f0aa48"
-					(reference "D702")
-					(unit 1)
-				)
+				(path "/3fe1c7d3-674a-46fe-b8de-0718a52fef91/a69e15f3-9c14-4aca-9191-41e586ada203/b77f0077-1926-4790-a8ae-2d9cb2a861f8"
+					(reference "D2802")
+					(unit 1)
+				)
+				(path "/3fe1c7d3-674a-46fe-b8de-0718a52fef91/a69e15f3-9c14-4aca-9191-41e586ada203/3b3a13db-6557-433d-96a5-218459e8b091"
+					(reference "D2602")
+					(unit 1)
+				)
+				(path "/3fe1c7d3-674a-46fe-b8de-0718a52fef91/a69e15f3-9c14-4aca-9191-41e586ada203/cbcba9a5-81e5-4be6-bbd1-91127981b75d"
+					(reference "D2702")
+					(unit 1)
+				)

Commit message: Many exiting news
Parts:
- removed R2801: 3k3, Resistor_SMD:R_0805_2012Metric_Pad1.20x1.40mm_HandSolder, symbol Device:R
Connections:
- net DCC0: no longer D2801.1 (K)
- net DCC1: now also D2801.2 (A)
- net at D2802.2 (A), R2802.2: now also D2801.1 (K)
Other:
- moved on the sheet: D2801, D2802, R2802
