File: kicad/xDuinoRailShield/rails_signal_extraction_analog.kicad_sch (KiCad schematic)
At the start: 2 parts

Commit message: Many exiting news
Parts:
- R401: renamed from R101; value 10K -> 10k; footprint (none) -> Resistor_SMD:R_0805_2012Metric_Pad1.20x1.40mm_HandSolder; OLI_ID (none) -> 10k_0805
- R402: renamed from R102; value 1K -> 1k; footprint (none) -> Resistor_SMD:R_0805_2012Metric_Pad1.20x1.40mm_HandSolder; OLI_ID (none) -> 1k_0805
Changed lines of the file:
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@@
 	(version 20231120)
 	(generator "eeschema")
-	(generator_version "7.99")
+	(generator_version "8.0")
 	(paper "A4")
 	(junction
@@
 		)
 	)
-	(hierarchical_label "GND"
+	(hierarchical_label "DCC1"
 		(shape input)
 		(at 39.37 67.31 180)
@@
 		(dnp no)
 		(fields_autoplaced yes)
-		(property "Reference" "R101"
+		(property "Reference" "R401"
 			(at 48.26 49.5299 0)
 			(effects
@@
 			)
 		)
-		(property "Value" "10K"
+		(property "Value" "10k"
 			(at 48.26 52.0699 0)
 			(effects
@@
 			)
 		)
-		(property "Footprint" ""
+		(property "Footprint" "Resistor_SMD:R_0805_2012Metric_Pad1.20x1.40mm_HandSolder"
 			(at 43.942 50.8 90)
 			(effects
@@
 			)
 		)
+		(property "OLI_ID" "10k_0805"
+			(at 45.72 50.8 0)
+			(effects
+				(font
+					(size 1.27 1.27)
+				)
+				(hide yes)
+			)
+		)
 		(pin "1"
 		)
@@
 		)
 		(instances
+			(project "xDuinoRail-Breakout-Railcom8x50"
+				(path "/3fe1c7d3-674a-46fe-b8de-0718a52fef91/de132676-c05c-4510-b783-d0cc70736386"
+					(reference "R401")
+					(unit 1)
+				)
+			)
 			(project "rails_signal_extraction_analog"
 				(path "/fcccac48-6e6b-491c-b569-290c1829c6bd"
@@
 		(dnp no)
 		(fields_autoplaced yes)
-		(property "Reference" "R102"
+		(property "Reference" "R402"
 			(at 48.26 59.6899 0)
 			(effects
@@
 			)
 		)
-		(property "Value" "1K"
+		(property "Value" "1k"
 			(at 48.26 62.2299 0)
 			(effects
@@
 			)
 		)
-		(property "Footprint" ""
+		(property "Footprint" "Resistor_SMD:R_0805_2012Metric_Pad1.20x1.40mm_HandSolder"
 			(at 43.942 60.96 90)
 			(effects
@@
 			)
 		)
+		(property "OLI_ID" "1k_0805"
+			(at 45.72 60.96 0)
+			(effects
+				(font
+					(size 1.27 1.27)
+				)
+				(hide yes)
+			)
+		)
 		(pin "1"
 		)
@@
 		)
 		(instances
+			(project "xDuinoRail-Breakout-Railcom8x50"
+				(path "/3fe1c7d3-674a-46fe-b8de-0718a52fef91/de132676-c05c-4510-b783-d0cc70736386"
+					(reference "R402")
+					(unit 1)
+				)
+			)
 			(project "rails_signal_extraction_analog"
 				(path "/fcccac48-6e6b-491c-b569-290c1829c6bd"
@@
 		(dnp no)
 		(fields_autoplaced yes)
-		(property "Reference" "#PWR0601"
+		(property "Reference" "#PWR0401"
 			(at 45.72 74.93 0)
 			(effects
@@
 		)
 		(instances
+			(project "xDuinoRail-Breakout-Railcom8x50"
+				(path "/3fe1c7d3-674a-46fe-b8de-0718a52fef91/de132676-c05c-4510-b783-d0cc70736386"
+					(reference "#PWR0401")
+					(unit 1)
+				)
+			)
 			(project "xDuinoRailShield"
 				(path "/e63e39d7-6ac0-4ffd-8aa3-1841a4541b55/f59f9ae7-6afc-4bf7-ac97-b34cf3a86d49"
@@
 		)
 	)
-	(sheet_instances
-		(path "/"
-			(page "1")
-		)
-	)
