File: kicad/xDuinoRailShield/rails_signal_extraction_dcc.kicad_sch (KiCad schematic)
At the start: 11 parts, among them Q1 T2N7002BK, U301 6N137, U302 EL817

Commit message: More refactoring
Parts:
- added R307: 10k, Resistor_SMD:R_0805_2012Metric_Pad1.20x1.40mm_HandSolder, symbol Device:R
- R5: value 22k -> 10k; footprint Resistor_SMD:R_0402_1005Metric_Pad0.72x0.64mm_HandSolder -> Resistor_SMD:R_0805_2012Metric_Pad1.20x1.40mm_HandSolder; LCSC C17560 -> C25744
Connections:
- net DCC0: no longer R5.1
- net DCC1: now also R5.1
- net DCC_MM_SIGNAL: now also R307.2; no longer R5.2
- new net: R307.1, R5.2
Changed lines of the file:
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@@
 	(wire
 		(pts
-			(xy 175.26 110.49) (xy 189.23 110.49)
+			(xy 175.26 110.49) (xy 176.53 110.49)
 		)
 		(stroke
@@
 		(pts
 			(xy 173.99 53.34) (xy 182.88 53.34)
+		)
+		(stroke
+			(width 0)
+			(type default)
+		)
+	)
+	(wire
+		(pts
+			(xy 184.15 110.49) (xy 189.23 110.49)
 		)
 		(stroke
@@
 		)
 	)
-	(label "DCC0"
+	(label "DCC1"
 		(at 154.94 110.49 0)
 		(fields_autoplaced yes)
@@
 				)
 			)
-			(project "xDuinoRailShield"
+			(project "xDuinoRailSwitch"
 				(path "/e63e39d7-6ac0-4ffd-8aa3-1841a4541b55/b84a333b-f29e-43df-b84d-edef752a64aa"
 					(reference "R304")
@@
 		)
 		(instances
-			(project "xDuinoRailShield"
+			(project "xDuinoRailSwitch"
 				(path "/e63e39d7-6ac0-4ffd-8aa3-1841a4541b55/b84a333b-f29e-43df-b84d-edef752a64aa"
 					(reference "#PWR0302")
@@
 				)
 			)
-			(project "xDuinoRailShield"
+			(project "xDuinoRailSwitch"
 				(path "/e63e39d7-6ac0-4ffd-8aa3-1841a4541b55/b84a333b-f29e-43df-b84d-edef752a64aa"
 					(reference "Q301")
@@
 		)
 		(instances
-			(project "xDuinoRailShield"
+			(project "xDuinoRailSwitch"
 				(path "/e63e39d7-6ac0-4ffd-8aa3-1841a4541b55/b84a333b-f29e-43df-b84d-edef752a64aa"
 					(reference "D301")
@@
 		)
 		(instances
-			(project "xDuinoRailShield"
+			(project "xDuinoRailSwitch"
 				(path "/e63e39d7-6ac0-4ffd-8aa3-1841a4541b55/b84a333b-f29e-43df-b84d-edef752a64aa"
 					(reference "#PWR0301")
@@
 		)
 		(instances
-			(project "xDuinoRailShield"
+			(project "xDuinoRailSwitch"
 				(path "/e63e39d7-6ac0-4ffd-8aa3-1841a4541b55/b84a333b-f29e-43df-b84d-edef752a64aa"
 					(reference "R303")
@@
 		)
 		(instances
-			(project "xDuinoRailShield"
+			(project "xDuinoRailSwitch"
 				(path "/e63e39d7-6ac0-4ffd-8aa3-1841a4541b55/b84a333b-f29e-43df-b84d-edef752a64aa"
 					(reference "#PWR0303")
+					(unit 1)
+				)
+			)
+		)
+	)
+	(symbol
+		(lib_id "Device:R")
+		(at 180.34 110.49 90)
+		(unit 1)
+		(exclude_from_sim no)
+		(in_bom no)
+		(on_board yes)
+		(dnp no)
+		(fields_autoplaced yes)
+		(property "Reference" "R307"
+			(at 180.34 104.14 90)
+			(effects
+				(font
+					(size 1.27 1.27)
+				)
+			)
+		)
+		(property "Value" "10k"
+			(at 180.34 106.68 90)
+			(effects
+				(font
+					(size 1.27 1.27)
+				)
+			)
+		)
+		(property "Footprint" "Resistor_SMD:R_0805_2012Metric_Pad1.20x1.40mm_HandSolder"
+			(at 180.34 112.268 90)
+			(effects
+				(font
+					(size 1.27 1.27)
+				)
+				(hide yes)
+			)
+		)
+		(property "Datasheet" "~"
+			(at 180.34 110.49 0)
+			(effects
+				(font
+					(size 1.27 1.27)
+				)
+				(hide yes)
+			)
+		)
+		(property "Description" "Resistor"
+			(at 180.34 110.49 0)
+			(effects
+				(font
+					(size 1.27 1.27)
+				)
+				(hide yes)
+			)
+		)
+		(property "LCSC" "C25744"
+			(at 180.34 110.49 0)
+			(effects
+				(font
+					(size 1.27 1.27)
+				)
+				(hide yes)
+			)
+		)
+		(property "Field-1" ""
+			(at 180.34 110.49 0)
+			(effects
+				(font
+					(size 1.27 1.27)
+				)
+				(hide yes)
+			)
+		)
+		(pin "1"
+		)
+		(pin "2"
+		)
+		(instances
+			(project "xDuinoRailSwitch"
+				(path "/e63e39d7-6ac0-4ffd-8aa3-1841a4541b55/b84a333b-f29e-43df-b84d-edef752a64aa"
+					(reference "R307")
 					(unit 1)
 				)
@@
 				)
 			)
-			(project "xDuinoRailShield"
+			(project "xDuinoRailSwitch"
 				(path "/e63e39d7-6ac0-4ffd-8aa3-1841a4541b55/b84a333b-f29e-43df-b84d-edef752a64aa"
 					(reference "#PWR0305")
@@
 		)
 		(instances
-			(project "xDuinoRailShield"
+			(project "xDuinoRailSwitch"
 				(path "/e63e39d7-6ac0-4ffd-8aa3-1841a4541b55/b84a333b-f29e-43df-b84d-edef752a64aa"
 					(reference "#PWR0304")
@@
 		)
 		(instances
-			(project "xDuinoRailShield"
+			(project "xDuinoRailSwitch"
 				(path "/e63e39d7-6ac0-4ffd-8aa3-1841a4541b55/b84a333b-f29e-43df-b84d-edef752a64aa"
 					(reference "U302")
@@
 		)
 		(instances
-			(project "xDuinoRailShield"
+			(project "xDuinoRailSwitch"
 				(path "/e63e39d7-6ac0-4ffd-8aa3-1841a4541b55/b84a333b-f29e-43df-b84d-edef752a64aa"
 					(reference "C301")
@@
 				)
 			)
-			(project "xDuinoRailShield"
+			(project "xDuinoRailSwitch"
 				(path "/e63e39d7-6ac0-4ffd-8aa3-1841a4541b55/b84a333b-f29e-43df-b84d-edef752a64aa"
 					(reference "R305")
@@
 		)
 		(instances
-			(project "xDuinoRailShield"
+			(project "xDuinoRailSwitch"
 				(path "/e63e39d7-6ac0-4ffd-8aa3-1841a4541b55/b84a333b-f29e-43df-b84d-edef752a64aa"
 					(reference "R302")
@@
 			)
 		)
-		(property "Value" "22k"
+		(property "Value" "10k"
 			(at 171.45 106.68 90)
 			(effects
@@
 			)
 		)
-		(property "Footprint" "Resistor_SMD:R_0402_1005Metric_Pad0.72x0.64mm_HandSolder"
+		(property "Footprint" "Resistor_SMD:R_0805_2012Metric_Pad1.20x1.40mm_HandSolder"
 			(at 171.45 112.268 90)
 			(effects
@@
 			)
 		)
-		(property "LCSC" "C17560"
+		(property "LCSC" "C25744"
 			(at 171.45 110.49 0)
 			(effects
@@
 				)
 			)
-			(project "xDuinoRailShield"
+			(project "xDuinoRailSwitch"
 				(path "/e63e39d7-6ac0-4ffd-8aa3-1841a4541b55/b84a333b-f29e-43df-b84d-edef752a64aa"
 					(reference "R306")
@@
 		)
 		(instances
-			(project "xDuinoRailShield"
+			(project "xDuinoRailSwitch"
 				(path "/e63e39d7-6ac0-4ffd-8aa3-1841a4541b55/b84a333b-f29e-43df-b84d-edef752a64aa"
 					(reference "R301")
@@
 		)
 		(instances
-			(project "xDuinoRailShield"
+			(project "xDuinoRailSwitch"
 				(path "/e63e39d7-6ac0-4ffd-8aa3-1841a4541b55/b84a333b-f29e-43df-b84d-edef752a64aa"
 					(reference "U301")

Commit message: More stuff
Parts:
- renumbered C301 to C2101, D301 to D2101, R301 to R2101, R302 to R2102, R303 to R2103, R5 to R2106, R307 to R2107, U301 to U2101, U302 to U2102

Commit message: Many exiting news
Parts:
- added R308: 10k, Resistor_SMD:R_0805_2012Metric_Pad1.20x1.40mm_HandSolder, symbol Device:R
- R1, R2: value 6k8 -> 10k; OLI_ID (none) -> 10k_0805
- R301: renamed from R2101; OLI_ID (none) -> 1k3_0805
- R302: renamed from R2102; OLI_ID (none) -> 220R_0805
- R303: renamed from R2103; value 5k -> 10k; OLI_ID (none) -> 10k_0805
- R306: renamed from R2106; OLI_ID (none) -> 10k_0805; now in the parts list
- R307: renamed from R2107; OLI_ID (none) -> 10k_0805; now in the parts list
- U301: renamed from U2101; OLI_ID (none) -> 6N137_SMD-6P
- U302: renamed from U2102; OLI_ID (none) -> EL817_SMD-4P
- renumbered C2101 to C301, D2101 to D301
Connections:
- net DCC_MM_SIGNAL: now also R308.1
- net +5V renamed +3v3
- net +3v3: now also R308.2
Other:
- moved on the sheet: C301, D301, R303
