File: kicad/xDuinoRailShield/rails_signal_feedback_dcc-railcom-8x50.kicad_sch (KiCad schematic)
At the start: 15 parts, among them Q401 S8050, Q402 S8550, Q403 S8550, Q404 S8050

Commit message: More stuff
Parts:
- removed TP101, TP102, TP103, TP104: TestPoint, TestPoint:TestPoint_Pad_D2.0mm, symbol Connector:TestPoint
- added D402: LED, LED_SMD:LED_0603_1608Metric_Pad1.05x0.95mm_HandSolder, symbol Device:LED
- added J401: Conn_01x05, Connector_PinHeader_2.54mm:PinHeader_1x05_P2.54mm_Vertical, symbol Connector_Generic:Conn_01x05
- added R406: 100R, Resistor_SMD:R_0805_2012Metric_Pad1.20x1.40mm_HandSolder, symbol Device:R
- D401: OLI_ID (none) -> 1N4148W_SOD-123
- JP401: value J_EnableRailcom -> SolderJumper_2_Bridged; footprint Jumper:SolderJumper-2_P1.3mm_Bridged_RoundedPad1.0x1.5mm -> Jumper:SolderJumper-2_P1.3mm_Bridged_Pad1.0x1.5mm
- Q401, Q404: OLI_ID (none) -> S8050_SOT-23
- Q402, Q403: OLI_ID (none) -> S8550_SOT-23
- R404: renamed from R9; OLI_ID (none) -> 10k_0805
- R405: renamed from R7; OLI_ID (none) -> 10k_0805
- renumbered R405 to R401, R404 to R402, R406 to R403
Connections:
- net GND: now also D402.1 (K), J401.5 (Pin_5)
- net RAILCOM_DATA: now also JP401.2 (B), J401.1 (Pin_1)
- net RC_CURR: now also J401.2 (Pin_2)
- net RC_FB_IN: now also J401.3 (Pin_3)
- net RC_ON_OFF: now also J401.4 (Pin_4)
- net RC_SIGNAL: now also Q402.3 (C); no longer JP401.2 (B)
- net at JP401.1 (A): now also R406.1; no longer Q402.3 (C)
- new net: D402.2 (A), R406.2

Commit message: Neue Breakouts
Parts:
- removed D402: LED, LED_SMD:LED_0603_1608Metric_Pad1.05x0.95mm_HandSolder, symbol Device:LED
- removed JP401: SolderJumper_2_Bridged, Jumper:SolderJumper-2_P1.3mm_Bridged_Pad1.0x1.5mm, symbol Jumper:SolderJumper_2_Bridged
- removed R406: 100R, Resistor_SMD:R_0805_2012Metric_Pad1.20x1.40mm_HandSolder, symbol Device:R
- J401: now not fitted; now left out of the parts list
- R401, R402, R403: OLI_ID (none) -> 10R_0805

Commit message: Many exiting news
Parts:
- J201: renamed from J401; footprint Connector_PinHeader_2.54mm:PinHeader_1x05_P2.54mm_Vertical -> Connector_Wire:SolderWire-0.5sqmm_1x05_P4.6mm_D0.9mm_OD2.1mm_Relief
- renumbered D401 to D201, Q401 to Q201, Q402 to Q202, Q403 to Q203, Q404 to Q204, R401 to R201, R402 to R202, R403 to R203, R404 to R204, R405 to R205
Connections:
- net RAILCOM_DATA: no longer J201.1 (Pin_1)
- net RC_SIGNAL: now also J201.1 (Pin_1)
- net 15R: now reaches R201.2, R202.2, R203.1
Changed lines of the file:
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@@
+	(wire
+		(pts
+			(xy 158.75 52.07) (xy 177.8 52.07)
+		)
+		(stroke
+			(width 0)
+			(type default)
+		)
+	)
 	(wire
 		(pts
@@
 	(wire
 		(pts
-			(xy 162.56 50.8) (xy 158.75 50.8)
-		)
-		(stroke
-			(width 0)
-			(type default)
-		)
-	)
-	(wire
-		(pts
 			(xy 68.58 91.44) (xy 71.12 91.44)
 		)
@@
 		(pts
 			(xy 68.58 102.87) (xy 60.96 102.87)
-		)
-		(stroke
-			(width 0)
-			(type default)
-		)
-	)
-	(wire
-		(pts
-			(xy 158.75 50.8) (xy 158.75 52.07)
 		)
 		(stroke
@@
 		)
 	)
+	(label "15R"
+		(at 62.23 45.72 0)
+		(fields_autoplaced yes)
+		(effects
+			(font
+				(size 1.27 1.27)
+			)
+			(justify left bottom)
+		)
+	)
 	(label "DCC0"
 		(at 44.45 111.76 0)
@@
 			)
 			(justify left bottom)
+		)
+	)
+	(label "RC_SIGNAL"
+		(at 177.8 52.07 180)
+		(fields_autoplaced yes)
+		(effects
+			(font
+				(size 1.27 1.27)
+			)
+			(justify right bottom)
 		)
 	)
@@
 		(shape input)
 		(at 130.81 95.25 0)
-		(fields_autoplaced yes)
-		(effects
-			(font
-				(size 1.27 1.27)
-			)
-			(justify left)
-		)
-	)
-	(hierarchical_label "RAILCOM_DATA"
-		(shape input)
-		(at 162.56 50.8 0)
 		(fields_autoplaced yes)
 		(effects
@@
 		(on_board yes)
 		(dnp no)
-		(property "Reference" "Q403"
+		(property "Reference" "Q203"
 			(at 91.44 58.42 0)
 			(effects
@@
 		)
 		(instances
-			(project "xDuinoRail-Breakout-Railcom8x50"
-				(path "/3fe1c7d3-674a-46fe-b8de-0718a52fef91/2953c156-b0e9-4c50-bb04-afd737c2b019"
-					(reference "Q403")
+			(project "xDuinoRail-Breakout-RailcomDetect"
+				(path "/3fe1c7d3-674a-46fe-b8de-0718a52fef91/f540c576-7d0b-4da2-8920-e9aaabc190c1"
+					(reference "Q203")
 					(unit 1)
 				)
@@
 		(on_board yes)
 		(dnp no)
-		(property "Reference" "R401"
+		(property "Reference" "R201"
 			(at 57.15 49.53 0)
 			(effects
@@
 		)
 		(instances
-			(project "xDuinoRail-Breakout-Railcom8x50"
-				(path "/3fe1c7d3-674a-46fe-b8de-0718a52fef91/2953c156-b0e9-4c50-bb04-afd737c2b019"
-					(reference "R401")
+			(project "xDuinoRail-Breakout-RailcomDetect"
+				(path "/3fe1c7d3-674a-46fe-b8de-0718a52fef91/f540c576-7d0b-4da2-8920-e9aaabc190c1"
+					(reference "R201")
 					(unit 1)
 				)
@@
 		(on_board yes)
 		(dnp no)
-		(property "Reference" "Q402"
+		(property "Reference" "Q202"
 			(at 68.58 66.04 0)
 			(effects
@@
 		)
 		(instances
-			(project "xDuinoRail-Breakout-Railcom8x50"
-				(path "/3fe1c7d3-674a-46fe-b8de-0718a52fef91/2953c156-b0e9-4c50-bb04-afd737c2b019"
-					(reference "Q402")
+			(project "xDuinoRail-Breakout-RailcomDetect"
+				(path "/3fe1c7d3-674a-46fe-b8de-0718a52fef91/f540c576-7d0b-4da2-8920-e9aaabc190c1"
+					(reference "Q202")
 					(unit 1)
 				)
@@
 		(on_board yes)
 		(dnp no)
-		(property "Reference" "R402"
+		(property "Reference" "R202"
 			(at 68.58 49.53 0)
 			(effects
@@
 		)
 		(instances
-			(project "xDuinoRail-Breakout-Railcom8x50"
-				(path "/3fe1c7d3-674a-46fe-b8de-0718a52fef91/2953c156-b0e9-4c50-bb04-afd737c2b019"
-					(reference "R402")
+			(project "xDuinoRail-Breakout-RailcomDetect"
+				(path "/3fe1c7d3-674a-46fe-b8de-0718a52fef91/f540c576-7d0b-4da2-8920-e9aaabc190c1"
+					(reference "R202")
 					(unit 1)
 				)
@@
 		(dnp no)
 		(fields_autoplaced yes)
-		(property "Reference" "#PWR0402"
+		(property "Reference" "#PWR0202"
 			(at 125.73 104.14 0)
 			(effects
@@
 		)
 		(instances
-			(project "xDuinoRail-Breakout-Railcom8x50"
-				(path "/3fe1c7d3-674a-46fe-b8de-0718a52fef91/2953c156-b0e9-4c50-bb04-afd737c2b019"
-					(reference "#PWR0402")
+			(project "xDuinoRail-Breakout-RailcomDetect"
+				(path "/3fe1c7d3-674a-46fe-b8de-0718a52fef91/f540c576-7d0b-4da2-8920-e9aaabc190c1"
+					(reference "#PWR0202")
 					(unit 1)
 				)
@@
 		(on_board yes)
 		(dnp no)
-		(property "Reference" "R403"
+		(property "Reference" "R203"
 			(at 77.47 43.18 0)
 			(effects
@@
 		)
 		(instances
-			(project "xDuinoRail-Breakout-Railcom8x50"
-				(path "/3fe1c7d3-674a-46fe-b8de-0718a52fef91/2953c156-b0e9-4c50-bb04-afd737c2b019"
-					(reference "R403")
+			(project "xDuinoRail-Breakout-RailcomDetect"
+				(path "/3fe1c7d3-674a-46fe-b8de-0718a52fef91/f540c576-7d0b-4da2-8920-e9aaabc190c1"
+					(reference "R203")
 					(unit 1)
 				)
@@
 		(on_board yes)
 		(dnp no)
-		(property "Reference" "Q401"
+		(property "Reference" "Q201"
 			(at 58.42 95.25 0)
 			(effects
@@
 		)
 		(instances
-			(project "xDuinoRail-Breakout-Railcom8x50"
-				(path "/3fe1c7d3-674a-46fe-b8de-0718a52fef91/2953c156-b0e9-4c50-bb04-afd737c2b019"
-					(reference "Q401")
+			(project "xDuinoRail-Breakout-RailcomDetect"
+				(path "/3fe1c7d3-674a-46fe-b8de-0718a52fef91/f540c576-7d0b-4da2-8920-e9aaabc190c1"
+					(reference "Q201")
 					(unit 1)
 				)
@@
 		(dnp no)
 		(fields_autoplaced yes)
-		(property "Reference" "R405"
+		(property "Reference" "R205"
 			(at 101.6 58.42 90)
 			(effects
@@
 		)
 		(instances
-			(project "xDuinoRail-Breakout-Railcom8x50"
-				(path "/3fe1c7d3-674a-46fe-b8de-0718a52fef91/2953c156-b0e9-4c50-bb04-afd737c2b019"
-					(reference "R405")
+			(project "xDuinoRail-Breakout-RailcomDetect"
+				(path "/3fe1c7d3-674a-46fe-b8de-0718a52fef91/f540c576-7d0b-4da2-8920-e9aaabc190c1"
+					(reference "R205")
 					(unit 1)
 				)
@@
 		(on_board yes)
 		(dnp no)
-		(property "Reference" "Q404"
+		(property "Reference" "Q204"
 			(at 115.57 96.52 0)
 			(effects
@@
 		)
 		(instances
-			(project "xDuinoRail-Breakout-Railcom8x50"
-				(path "/3fe1c7d3-674a-46fe-b8de-0718a52fef91/2953c156-b0e9-4c50-bb04-afd737c2b019"
-					(reference "Q404")
+			(project "xDuinoRail-Breakout-RailcomDetect"
+				(path "/3fe1c7d3-674a-46fe-b8de-0718a52fef91/f540c576-7d0b-4da2-8920-e9aaabc190c1"
+					(reference "Q204")
 					(unit 1)
 				)
@@
 		(dnp no)
 		(fields_autoplaced yes)
-		(property "Reference" "#PWR0401"
+		(property "Reference" "#PWR0201"
 			(at 88.9 48.26 0)
 			(effects
@@
 		)
 		(instances
-			(project "xDuinoRail-Breakout-Railcom8x50"
-				(path "/3fe1c7d3-674a-46fe-b8de-0718a52fef91/2953c156-b0e9-4c50-bb04-afd737c2b019"
-					(reference "#PWR0401")
+			(project "xDuinoRail-Breakout-RailcomDetect"
+				(path "/3fe1c7d3-674a-46fe-b8de-0718a52fef91/f540c576-7d0b-4da2-8920-e9aaabc190c1"
+					(reference "#PWR0201")
 					(unit 1)
 				)
@@
 		(on_board yes)
 		(dnp no)
-		(property "Reference" "R404"
+		(property "Reference" "R204"
 			(at 90.17 97.79 90)
 			(effects
@@
 		)
 		(instances
-			(project "xDuinoRail-Breakout-Railcom8x50"
-				(path "/3fe1c7d3-674a-46fe-b8de-0718a52fef91/2953c156-b0e9-4c50-bb04-afd737c2b019"
-					(reference "R404")
+			(project "xDuinoRail-Breakout-RailcomDetect"
+				(path "/3fe1c7d3-674a-46fe-b8de-0718a52fef91/f540c576-7d0b-4da2-8920-e9aaabc190c1"
+					(reference "R204")
 					(unit 1)
 				)
@@
 		(on_board yes)
 		(dnp yes)
-		(property "Reference" "J401"
+		(property "Reference" "J201"
 			(at 151.13 55.8799 0)
 			(effects
@@
 			)
 		)
-		(property "Footprint" "Connector_PinHeader_2.54mm:PinHeader_1x05_P2.54mm_Vertical"
+		(property "Footprint" "Connector_Wire:SolderWire-0.5sqmm_1x05_P4.6mm_D0.9mm_OD2.1mm_Relief"
 			(at 153.67 57.15 0)
 			(effects
@@
 		)
 		(instances
-			(project "xDuinoRail-Breakout-Railcom8x50"
-				(path "/3fe1c7d3-674a-46fe-b8de-0718a52fef91/2953c156-b0e9-4c50-bb04-afd737c2b019"
-					(reference "J401")
+			(project "xDuinoRail-Breakout-RailcomDetect"
+				(path "/3fe1c7d3-674a-46fe-b8de-0718a52fef91/f540c576-7d0b-4da2-8920-e9aaabc190c1"
+					(reference "J201")
 					(unit 1)
 				)
@@
 		(on_board no)
 		(dnp yes)
-		(property "Reference" "D401"
+		(property "Reference" "D201"
 			(at 58.42 85.09 90)
 			(effects
@@
 		)
 		(instances
-			(project "xDuinoRail-Breakout-Railcom8x50"
-				(path "/3fe1c7d3-674a-46fe-b8de-0718a52fef91/2953c156-b0e9-4c50-bb04-afd737c2b019"
-					(reference "D401")
+			(project "xDuinoRail-Breakout-RailcomDetect"
+				(path "/3fe1c7d3-674a-46fe-b8de-0718a52fef91/f540c576-7d0b-4da2-8920-e9aaabc190c1"
+					(reference "D201")
 					(unit 1)
 				)
